File: PCB/Watch_V3/Watch_v3.kicad_pcb (KiCad board)
At the start: 2 copper layers, 84 parts, among them J1 USB_C_Receptacle_USB2.0_16P, J2 Screw_Terminal, J3 Peripheral, J4 OLED, J5 BN220, J6 Peripheral, J7 MAX30102, M1 Motor_DC, Q1 AO3401A, Q2 BC817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

Commit message: updating PCB_watchV3
Parts:
- removed BZ1: Buzzer, Buzzer_Beeper:Buzzer_12x9.5RM7.6
- removed R20: 2.2E, Resistor_SMD:R_01005_0402Metric
- added D7: SS34, Capacitor_SMD:ss34_DO, F.Cu at (138.1, 119.6)
- added LS1: CMT-8530S-SMT, Capacitor_SMD:CUI_CMT-8530S-SMT, B.Cu at (196.8, 76.5)
- added Q5: BC847, Package_TO_SOT_SMD:SOT-23, F.Cu at (81.5, 134.6)
- SW1, SW3: footprint Button_Switch_SMD:SW_Push_1P1T_NO_6x6mm_H9.5mm -> Button_Switch_SMD:SW_Tactile_SPST_NO_Straight_CK_PTS636Sx25SMTRLFS
- SW4, SW5, SW6, SW7, U3: moved to B.Cu
- moved SW6 195.9 mm to (204.3, 85.9), turned to 180 degrees
- moved SW7 194.6 mm to (204.3, 97.0), turned to 180 degrees
- moved SW1 185.6 mm to (200.4, 76.2), turned to 90 degrees
- moved Y1 182.7 mm to (195.8, 107.2), turned to 90 degrees
- moved U3 165.6 mm to (186.9, 101.9), turned to 180 degrees
- moved SW3 161.8 mm to (172.7, 75.9), turned to 90 degrees
- moved SW4 159.1 mm to (170.7, 85.9), turned to 180 degrees
- moved SW5 157.8 mm to (170.7, 97.0), turned to 180 degrees
- moved U4 155.2 mm to (187.3, 78.1)
- moved J4 149.6 mm to (182.9, 95.8), turned to 90 degrees
- moved U5 148.8 mm to (204.5, 90.2)
- moved J1 134.1 mm to (186.9, 112.8)
- moved U6 117.6 mm to (186.7, 101.6)
- moved J7 105.4 mm to (179.1, 91.5), turned to 90 degrees
- moved SW2 103.3 mm to (177.0, 108.6), turned to 90 degrees
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Routing:
- net GND: track 0.00 -> 31.8 mm
- net /Mode: track 0.00 -> 7.95 mm
- net /Down: track 0.00 -> 7.95 mm
- net /Up: track 0.00 -> 7.95 mm
- net /Select: track 0.00 -> 7.95 mm
Other:
- board outline added: 50 x 50 mm
- copper layers 2 -> 4
