File: PCB/Watch_V3/Watch_v3.kicad_pcb (KiCad board)
At the start: 4 copper layers, 98 parts, among them J1 USB_C_Receptacle_USB2.0_16P, J2 Screw_Terminal, J3 Peripheral, J4 OLED, J5 BN220, J6 Peripheral, J7 MAX30102, M1 Motor_DC, Q1 AO3401A, Q2 BC817, Q3 BC817, Q4 SI2302, Q5 BC847, SW1 SW_DPST_x2, SW2 SW_SPDT, SW3 SW_DPST_x2, SW4 Select, SW5 Mode, SW6 Up, SW7 Down, U1 AP2112K-3.3, U2 AP2112K-3.3, U3 TP4056, U4 ESP32-WROOM-32D, U5 CP2102N-Axx-xQFN28, U6 MPU-6050

Commit message: updating watch_v3
Parts:
- removed R28: 0, Resistor_SMD:R_0201_0603Metric
- added R34: 0, Resistor_SMD:R_0402_1005Metric, F.Cu at (25.0, 59.3)
- added R39: 0, Resistor_SMD:R_0402_1005Metric, F.Cu at (25.0, 69.3)
- C1, C10, C11, C12, C13, C14, C15, C16, C17, C18, C19, C2, C20, C22, C23, C25, C26, C27, C28, C3, C4, C5, C6, C7, C8, C9: footprint Capacitor_SMD:C_0603_1608Metric -> Capacitor_SMD:C_0402_1005Metric
- D2, D3, D4, D5, D6: footprint LED_SMD:LED_0603_1608Metric -> LED_SMD:LED_0402_1005Metric
- J1: footprint Connector_USB:USB_C_Receptacle_HCTL_HC-TYPE-C-16P-01A -> Connector_USB:USB_C_Receptacle_GCT_USB4105-xx-A_16P_TopMnt_Horizontal
- R1, R10, R11, R12, R13, R14, R15, R16, R17, R18, R19, R2, R20, R21, R22, R23, R24, R25, R26, R27, R29, R3, R32, R33, R35, R36, R37, R38, R4, R5, R6, R7, R8, R9: footprint Resistor_SMD:R_0201_0603Metric -> Resistor_SMD:R_0402_1005Metric
- R30, R31: value 1K -> 220E; footprint Resistor_SMD:R_0201_0603Metric -> Resistor_SMD:R_0402_1005Metric
- moved U4 120.5 mm to (36.7, 47.3)
- moved J7 85.6 mm to (40.3, 60.7)
- moved SW2 83.9 mm to (15.9, 77.8)
- moved C7 83.4 mm to (27.9, 71.1)
- moved D2 82.5 mm to (73.7, 16.8)
- moved D6 79.2 mm to (73.7, 24.8)
- moved D3 78.1 mm to (73.7, 18.8)
- moved U5 77.5 mm to (51.1, 73.0)
- moved J1 77.2 mm to (67.3, 52.6)
- moved C14 76.4 mm to (30.8, 71.1)
- moved D5 74.5 mm to (73.7, 22.8)
- moved Q5 73.4 mm to (45.1, 73.9)
- moved C21 73.0 mm to (33.7, 71.1)
- moved C6 72.5 mm to (27.9, 69.2)
- moved R32 72.1 mm to (22.1, 71.3)
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Connections:
- C2 pad 2: VBUS -> Net-(Q1-D)
- D1 pad C: VBUS -> Net-(Q1-D)
- J2 pad 1: Net-(J2-Pin_1) -> +BATT
- J6 pad 2: +3.3V -> Net-(J6-Pin_2)
- Q1 pad 3: VBUS -> Net-(Q1-D)
Other:
- copper layers 4 -> 2

Commit message: remote_v3
Parts:
- added J8: ICSP, Button_Switch_SMD:solder_pad_4, F.Cu at (78.4, 43.7)
Changed lines of the file:
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@@
     )
+  )
+  (footprint "Button_Switch_SMD:solder_pad_4" (layer "F.Cu")
+    (at 78.426 43.694)
+    (property "Sheetfile" "Watch_v3.kicad_sch")
+    (property "Sheetname" "")
+    (property "ki_description" "Generic connector, single row, 01x04, script generated")
+    (property "ki_keywords" "connector")
+    (attr smd)
+    (fp_text reference "J8" (at 0 -0.5 unlocked) (layer "F.SilkS")
+        (effects (font (size 1 1) (thickness 0.1)))
+    )
+    (fp_text value "ICSP" (at 0 1 unlocked) (layer "F.Fab")
+        (effects (font (size 1 1) (thickness 0.15)))
+    )
+    (fp_text user "${REFERENCE}" (at 0 2.5 unlocked) (layer "F.Fab")
+        (effects (font (size 1 1) (thickness 0.15)))
+    )
+    (pad "1" smd circle (at -2.55 -2.8) (size 1.5 1.5) (layers "F.Cu" "F.Paste" "F.Mask")
+      (net 1 "GND") (pinfunction "Pin_1") (pintype "passive"))
+    (pad "2" smd circle (at -0.85 -2.8) (size 1.5 1.5) (layers "F.Cu" "F.Paste" "F.Mask")
+      (net 17 "/TX") (pinfunction "Pin_2") (pintype "passive"))
+    (pad "3" smd circle (at 0.9 -2.8) (size 1.5 1.5) (layers "F.Cu" "F.Paste" "F.Mask")
+      (net 15 "/RX") (pinfunction "Pin_3") (pintype "passive"))
+    (pad "4" smd circle (at 2.6 -2.8) (size 1.5 1.5) (layers "F.Cu" "F.Paste" "F.Mask")
+      (net 2 "+5V") (pinfunction "Pin_4") (pintype "passive"))
   )
   (footprint "Resistor_SMD:R_0402_1005Metric" (layer "F.Cu")

Commit message: remote_v2 update
Parts:
- moved D4 155.9 mm to (76.9, 176.7)
- moved D2 155.9 mm to (76.9, 172.7)
- moved D3 155.9 mm to (76.9, 174.7)
- moved D5 155.9 mm to (76.9, 178.7)
- moved D6 155.9 mm to (76.9, 180.7)
- moved J8 145.9 mm to (24.0, 179.1)
- moved J1 124.4 mm to (69.3, 177.0)
- moved U1 113.6 mm to (80.9, 173.9)
- moved U2 113.6 mm to (80.9, 178.4)
- moved U3 111.1 mm to (38.0, 179.9)
- moved J3 109.3 mm to (24.0, 164.7)
- moved J6 109.3 mm to (24.0, 174.3)
- moved J5 109.3 mm to (24.0, 169.5)
- moved U5 105.0 mm to (51.0, 178.1)
- moved C10 104.4 mm to (51.7, 165.6)
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
Commit message: update remote_v2
Parts:
- moved SW3 6.51 mm to (72.4, 132.1)
- moved R1 6.51 mm to (32.0, 167.7)
- moved R2 6.51 mm to (32.0, 169.7)
- moved R3 6.51 mm to (32.0, 171.7)
- moved R4 6.51 mm to (32.0, 173.7)
- moved R6 6.51 mm to (32.0, 177.7)
- moved R7 6.51 mm to (32.0, 179.7)
- moved C12 6.51 mm to (49.4, 175.6)
- moved C13 6.51 mm to (49.4, 177.6)
- moved C14 6.51 mm to (49.4, 179.6)
- moved C15 6.51 mm to (52.3, 167.7)
- moved C19 6.51 mm to (52.3, 175.6)
- moved C20 6.51 mm to (52.3, 177.6)
- moved C21 6.51 mm to (52.3, 179.6)
- moved C8 6.51 mm to (49.4, 167.7)
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
Commit message: update watch_v3
Parts:
- J2, LS1, M1, Q4, Q5, U3, U6: moved to B.Cu
- R7: value 1K -> 1.2K
- SW4: value Select -> Mode
- SW5: value Mode -> Down
- SW6: value Up -> Select
- SW7: value Down -> Up
- moved J5 185.4 mm to (172.0, 67.0), turned to 90 degrees
- moved J6 182.8 mm to (171.9, 76.2), turned to 90 degrees
- moved R23 181.4 mm to (166.2, 51.6), turned to -90 degrees
- moved Q5 179.7 mm to (157.1, 57.3), turned to 180 degrees
- moved R13 178.7 mm to (165.9, 54.1), turned to 90 degrees
- moved R8 168.7 mm to (164.8, 77.7)
- moved C27 168.6 mm to (169.3, 51.5), turned to 90 degrees
- moved C8 165.3 mm to (169.4, 54.1), turned to 90 degrees
- moved R26 164.6 mm to (167.2, 64.3)
- moved Q3 164.3 mm to (161.9, 82.5)
- moved Q2 163.9 mm to (161.9, 78.7)
- moved U3 162.2 mm to (165.2, 88.4), turned to 180 degrees
- moved R21 160.7 mm to (139.6, 51.3), turned to -90 degrees
- moved R39 157.5 mm to (167.7, 80.6), turned to 90 degrees
- moved R9 156.1 mm to (164.8, 81.3)
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Routing:
- net GND: track 0.00 -> 190.1 mm, vias 0 -> 12
- net +3.3V: track 0.00 -> 75.3 mm, vias 0 -> 5
- net /SCL: track 0.00 -> 52.0 mm, vias 0 -> 4
- net /Up: track 0.00 -> 51.6 mm, vias 0 -> 8
- net /EN: track 0.00 -> 46.7 mm, vias 0 -> 3
- net /SDA: track 0.00 -> 42.1 mm, vias 0 -> 2
- net VBUS: track 0.00 -> 42.1 mm, vias 0 -> 2
- net /Down: track 0.00 -> 41.2 mm, vias 0 -> 2
- net /ADC_Batt: track 0.00 -> 33.5 mm, vias 0 -> 4
- net /IO0: track 0.00 -> 33.5 mm, vias 0 -> 1
- net /motor: track 0.00 -> 29.3 mm, vias 0 -> 5
- net /TX: track 0.00 -> 26.3 mm, vias 0 -> 1
- net /DTR: track 0.00 -> 21.4 mm, vias 0 -> 4
- net /RX: track 0.00 -> 21.3 mm, vias 0 -> 2
- net /RTS: track 0.00 -> 18.3 mm, vias 0 -> 2
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Other:
- board outline added: 39.1 x 63.2 mm
- board text added: "C1"
- board text added: "ESP32-WROOM-32D"
- board text added: "SW1"
- board text added: "SW3"

Commit message: update watch_v3
Parts:
- C22, C23, D7, R18, R29, R33, R35, R36: moved to B.Cu
- moved J8 166.7 mm to (172.0, 89.5), turned to 90 degrees
- moved J3 163.0 mm to (172.0, 81.9), turned to 90 degrees
- moved R15 161.3 mm to (165.6, 67.2), turned to 90 degrees
- moved R14 158.6 mm to (167.7, 71.7), turned to -90 degrees
- moved R10 153.4 mm to (165.6, 69.5), turned to 90 degrees
- moved R11 153.1 mm to (165.3, 71.7), turned to 90 degrees
- moved R29 150.0 mm to (157.9, 63.5), turned to 180 degrees
- moved R7 148.8 mm to (166.1, 91.9)
- moved R6 148.7 mm to (162.5, 84.9)
- moved R37 146.6 mm to (165.6, 73.7), turned to 90 degrees
- moved R12 143.3 mm to (143.4, 64.4)
- moved R5 143.0 mm to (161.8, 91.9)
- moved R33 143.0 mm to (159.6, 83.5), turned to 180 degrees
- moved R32 142.5 mm to (159.1, 81.7), turned to -90 degrees
- moved C21 142.4 mm to (167.0, 77.7)
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Routing:
- net /Up: track 51.6 -> 3.12 mm, vias 8 -> 0
- net GND: track 190.1 -> 230.1 mm, vias 12 -> 14
- net /EN: track 46.7 -> 7.21 mm, vias 3 -> 2
- net /Down: track 41.2 -> 3.18 mm, vias 2 -> 0
- net /SCL: track 52.0 -> 14.8 mm, vias 4 -> 1
- net /motor: track 29.3 -> 0.00 mm, vias 5 -> 0
- net /SDA: track 42.1 -> 15.3 mm, vias 2 -> 1
- net /TX: track 26.3 -> 0.00 mm, vias 1 -> 0
- net +BATT: track 9.09 -> 30.5 mm, vias 1 -> 6
- net +5V: track 14.4 -> 32.0 mm, vias 0 -> 2
- net Net-(Q1-D): track 7.70 -> 22.7 mm, vias 2 -> 4
- net /Select: track 16.8 -> 3.65 mm, vias 1 -> 0
- net Net-(U4-VDD): track 0.00 -> 12.8 mm, vias 0 -> 3
- net +3.3V: track 75.3 -> 64.4 mm, vias 5 -> 8
- net Net-(U3-VCC): track 0.00 -> 9.79 mm, vias 0 -> 1
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
Commit message: update watch_v3
Parts:
- added G***: LOGO, Battery:xx, B.Cu at (163.9, 68.4)
- added G***: LOGO, Battery:robo2, B.Cu at (149.7, 58.9)
- C21: moved to B.Cu
- moved J3 37.9 mm to (135.2, 73.0)
- moved C21 11.2 mm to (157.4, 72.0)
- moved C18 0.63 mm to (167.3, 73.7)
- moved C20 0.10 mm to (166.9, 76.0)
- moved D6 0.05 mm to (166.5, 71.7)
Routing:
- net GND: track 230.1 -> 395.4 mm, vias 14 -> 203
- net +3.3V: track 64.4 -> 169.1 mm, vias 8 -> 24
- net /TX: track 0.00 -> 88.3 mm, vias 0 -> 16
- net /SDA: track 15.3 -> 80.4 mm, vias 1 -> 8
- net /SCL: track 14.8 -> 79.7 mm, vias 1 -> 11
- net /Up: track 3.12 -> 58.5 mm, vias 0 -> 10
- net /EN: track 7.21 -> 55.3 mm, vias 2 -> 9
- net /RX: track 27.0 -> 66.2 mm, vias 0 -> 6
- net /Down: track 3.18 -> 41.6 mm, vias 0 -> 2
- net Net-(J4-Pin_2): track 0.00 -> 36.2 mm, vias 0 -> 5
- net /Select: track 3.65 -> 33.6 mm, vias 0 -> 2
- net /motor: track 0.00 -> 28.3 mm, vias 0 -> 3
- net VBUS: track 36.0 -> 61.4 mm, vias 4 -> 10
- net /Mode: track 3.64 -> 26.2 mm, vias 0 -> 2
- net /27: track 0.00 -> 20.9 mm, vias 0 -> 4
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- added copper zone on B.Cu, net GND
- added copper zone on F.Cu, net GND
Other:
- board text added: "ARKA"
- board text added: "DHARMA ROBOFEST"
- board text added: "KRS"

Commit message: updating watch_v3
Parts:
- moved G*** 26.2 mm to (144.4, 85.9)
Routing:
- net /EN: track 55.3 -> 56.6 mm
- net GND: track 395.4 -> 394.7 mm, vias 203 -> 87
- net (no net): vias 6 -> 0
Other:
- board text added: "+"
- board text added: "-"
- board text added: "3.3"
- board text added: "5V"
- board text added: "Batt"
- board text added: "G"
- board text added: "G12"
- board text added: "G14"
- board text added: "G27"
- board text added: "M"
- board text added: "RX"
- board text added: "RX{dblquote}"
- board text added: "SCL"
- board text added: "SDA"
- board text added: "TX"
- board text added: "TX{dblquote}"
