File: PCB/Watch_V3/_autosave-Watch_v3.kicad_pcb (KiCad board)
At the start: 4 copper layers, 98 parts, among them J1 USB_C_Receptacle_USB2.0_16P, J2 Screw_Terminal, J3 Peripheral, J4 OLED, J5 BN220, J6 Peripheral, J7 MAX30102, M1 Motor_DC, Q1 AO3401A, Q2 BC817, Q3 BC817, Q4 SI2302, Q5 BC847, SW1 SW_DPST_x2, SW2 SW_SPDT, SW3 SW_DPST_x2, SW4 Select, SW5 Mode, SW6 Up, SW7 Down, U1 AP2112K-3.3, U2 AP2112K-3.3, U3 TP4056, U4 ESP32-WROOM-32D, U5 CP2102N-Axx-xQFN28, U6 MPU-6050

Commit message: updating watch_V3
Parts:
- J1: footprint Connector_USB:USB_C_Receptacle_HCTL_HC-TYPE-C-16P-01A -> Connector_USB:USB_C_Receptacle_GCT_USB4105-xx-A_16P_TopMnt_Horizontal

Commit message: updating watch_v3
Parts:
- removed R28: 0, Resistor_SMD:R_0201_0603Metric
- added R34: 0, Resistor_SMD:R_0402_1005Metric, F.Cu at (37.3, 69.9)
- added R39: 0, Resistor_SMD:R_0402_1005Metric, F.Cu at (37.3, 71.9)
- C1, C10, C11, C12, C13, C14, C15, C16, C17, C18, C19, C2, C20, C22, C23, C25, C26, C27, C28, C3, C4, C5, C6, C7, C8, C9: footprint Capacitor_SMD:C_0603_1608Metric -> Capacitor_SMD:C_0402_1005Metric
- D2, D3, D4, D5, D6: footprint LED_SMD:LED_0603_1608Metric -> LED_SMD:LED_0402_1005Metric
- LS1: moved to B.Cu
- R1, R10, R11, R12, R13, R14, R15, R16, R17, R18, R19, R2, R20, R21, R22, R23, R24, R25, R26, R27, R29, R3, R32, R33, R35, R36, R37, R38, R4, R5, R6, R7, R8, R9: footprint Resistor_SMD:R_0201_0603Metric -> Resistor_SMD:R_0402_1005Metric
- R30, R31: value 1K -> 220E; footprint Resistor_SMD:R_0201_0603Metric -> Resistor_SMD:R_0402_1005Metric
- moved J1 120.2 mm to (195.8, 112.2)
- moved J7 119.6 mm to (140.2, 96.0), turned to 90 degrees
- moved LS1 64.6 mm to (112.8, 95.4), turned to 180 degrees
- moved U4 45.4 mm to (195.4, 89.6)
- moved Q1 4.84 mm to (49.4, 121.2)
Connections:
- C2 pad 2: VBUS -> Net-(Q1-D)
- D1 pad C: VBUS -> Net-(Q1-D)
- J2 pad 1: Net-(J2-Pin_1) -> +BATT
- J6 pad 2: +3.3V -> Net-(J6-Pin_2)
- Q1 pad 3: VBUS -> Net-(Q1-D)
Other:
- board outline added: 87.9 x 50 mm
