File: PCB/Watch_V3/Watch_v3.kicad_sch (KiCad schematic)
At the start: 29 parts, among them J1 USB_C_Receptacle_USB2.0_16P, Q1 AO3401A, SW1 SW_DPST_x2, U1 AP2112K-3.3, U2 AP2112K-3.3, U3 AP2112K-3.3, U4 AP2112K-3.3

Commit message: update PCB_watchV3
Parts:
- removed U3, U4: AP2112K-3.3, Package_TO_SOT_SMD:SOT-23-5, symbol Regulator_Linear:AP2112K-3.3
- added BZ1: Buzzer, Buzzer_Beeper:Buzzer_12x9.5RM7.6, symbol Device:Buzzer
- added C17, C18, C19, C20, C21, C22, C25, C26, C27, C28: 0.1uF, Capacitor_SMD:C_0402_1005Metric, symbol Device:C
- added C23: 2.2nF, Capacitor_SMD:C_0402_1005Metric, symbol Device:C
- added D3, D4, D5, D6: LED, LED_SMD:LED_0402_1005Metric, symbol Device:LED
- added J2: Screw_Terminal, Button_Switch_SMD:solder_pad_batt, symbol Connector:Screw_Terminal_01x02
- added J3, J6: Peripheral, Button_Switch_SMD:solder_pad_4, symbol Connector:Conn_01x04_Pin
- added J4: OLED, Connector_PinHeader_2.54mm:PinHeader_1x04_P2.54mm_Vertical, symbol Connector:Conn_01x04_Pin
- added J5: BN220, Button_Switch_SMD:solder_pad_4, symbol Connector:Conn_01x04_Pin
- added J7: MAX30102, Connector_PinHeader_2.54mm:PinHeader_1x07_P2.54mm_Vertical, symbol Connector:Conn_01x07_Pin
- added M1: Motor_DC, Button_Switch_SMD:solder_motor, symbol Motor:Motor_DC
- added Q2, Q3: BC817, Package_TO_SOT_SMD:SOT-23, symbol Transistor_BJT:BC817
- added Q4: SI2302, SI2302:SOT23, symbol SI2302:SI2302
- added R10, R11: 150E, Resistor_SMD:R_01005_0402Metric, symbol Device:R
- added R12, R13, R14, R15, R16, R18, R19, R21, R22, R23, R24, R5, R6, R7, R8, R9: 1K, Resistor_SMD:R_01005_0402Metric, symbol Device:R
- added R17: 10K, Resistor_SMD:R_01005_0402Metric, symbol Device:R
- added R20: 2.2E, Resistor_SMD:R_01005_0402Metric, symbol Device:R
- added SW2: SW_SPDT, Button_Switch_THT:SW_Slide_1P2T_CK_OS102011MS2Q, symbol Switch:SW_SPDT
- added SW3: SW_DPST_x2, Button_Switch_SMD:SW_Push_1P1T_NO_6x6mm_H9.5mm, symbol Switch:SW_DPST_x2
- added SW4: Select, Button_Switch_SMD:SW_Push_1P1T_NO_6x6mm_H9.5mm, symbol Switch:SW_DPST_x2
- added SW5: Mode, Button_Switch_SMD:SW_Push_1P1T_NO_6x6mm_H9.5mm, symbol Switch:SW_DPST_x2
- added SW6: Up, Button_Switch_SMD:SW_Push_1P1T_NO_6x6mm_H9.5mm, symbol Switch:SW_DPST_x2
- added SW7: Down, Button_Switch_SMD:SW_Push_1P1T_NO_6x6mm_H9.5mm, symbol Switch:SW_DPST_x2
- added U3: TP4056, TP4056:SOP127P600X175-9N, symbol Amplifier_Audio:TP4056
- added U4: ESP32-WROOM-32D, RF_Module:ESP32-WROOM-32D, symbol RF_Module:ESP32-WROOM-32D
- added U5: CH340G, Package_SO:SOIC-16_3.9x9.9mm_P1.27mm, symbol Interface_USB:CH340G
- added U6: MPU-6050, Button_Switch_SMD:QFN50P400X400X95-24N, symbol MPU-6050:MPU-6050
- added Y1: 12M, Crystal:Crystal_HC49-4H_Vertical, symbol Device:Crystal
- C1, C10, C11, C12, C13, C14, C15, C16, C2, C3, C6, C7, C8, C9: footprint (none) -> Capacitor_SMD:C_0402_1005Metric
- C4, C5: value 0.1uF -> 22pF; footprint (none) -> Capacitor_SMD:C_0402_1005Metric
- D1: footprint SS34:DIOM7959X265N -> Capacitor_SMD:ss34_DO
- D2: footprint (none) -> LED_SMD:LED_0402_1005Metric
- J1: footprint (none) -> Connector_USB:USB_C_Receptacle_HCTL_HC-TYPE-C-16P-01A
- R1, R2, R3: footprint (none) -> Resistor_SMD:R_01005_0402Metric
- R4: value 150R -> 150E; footprint (none) -> Resistor_SMD:R_01005_0402Metric
- SW1: footprint (none) -> Button_Switch_SMD:SW_Push_1P1T_NO_6x6mm_H9.5mm
Connections:
- net +3.3V: now also C6.1, C9.2, C17.2, C18.2, C19.2, C20.2, C21.1, J4.2 (Pin_2), J5.4 (Pin_4), J6.2 (Pin_2), J7.1 (Pin_1), Q4.3, R10.1, R11.1, R12.2, R13.2, R14.2, R15.1, R21.2, R22.2, R23.2, R24.2, U4.2 (VDD), U5.16 (VCC), U5.4 (V3), U6.13 (VDD), U6.8 (VLOGIC)
- net +5V: now also D3.2 (A), D4.2 (A), U3.4 (VCC), U3.8 (CE)
- net +BATT: now also J2.1 (Pin_1), R16.1, U3.5 (BAT)
- net D+: now also U5.5 (UD+)
- net D-: now also U5.6 (UD-)
- net EN: now also C7.2, Q2.3 (C), R12.1, U4.3 (EN); no longer U1.3 (EN), U2.3 (EN)
- net GND: now also C5.1, C7.1, C8.1, C9.1, SW1.1 (A), BZ1.2 (-), C17.1, C18.1, C19.1, C20.1, C21.2, C22.2, C23.2, C25.1, C26.1, C27.1, C28.1, J2.2 (Pin_2), J4.1 (Pin_1), J5.1 (Pin_1), J6.1 (Pin_1), J7.7 (Pin_7), M1.2 (-), R17.2, R18.2, R7.1, SW3.1 (A), SW4.2 (B), SW5.2 (B), SW6.2 (B), SW7.2 (B), U3.3 (GND), U3.9 (EP), U4.1 (GND), U4.15 (GND), U4.38 (GND), U4.39 (GND), U5.1 (GND), U6.1 (CLKIN), U6.11 (FSYNC), U6.18 (GND); no longer C5.2, C7.2, C8.2, C9.2
- net VBUS: now also SW2.2 (B); no longer C4.1, C5.1, C6.1, C7.1, C8.1, C9.1, SW1.1 (A)
- new net: R7.2, U3.1 (TEMP), U3.2 (PROG)
- new net: R5.1, U3.6 (~{STDBY})
- new net: R6.1, U3.7 (~{CHRG})
- new net: Q3.1 (B), R9.1
- new net: D6.2 (A), R11.2
- new net: R19.1, SW2.1 (A)
- new net: M1.1 (+), Q4.2
- new net: D4.1 (K), R6.2
- new net: C5.2, U5.7 (XI), Y1.1
- new net: R18.1, U6.9 (AD0)
- new net: C4.1, U5.8 (XO), Y1.2
- new net: Q2.1 (B), R8.1
- new net: BZ1.1 (+), R20.2
- new net: D3.1 (K), R5.2
- new net: D5.2 (A), R10.2
- new net: C23.1, U6.20 (CPOUT)
- new net: C22.1, U6.10 (REGOUT)
- new net: U6.14 (NC), U6.15 (NC), U6.16 (NC), U6.17 (NC), U6.2 (NC), U6.3 (NC), U6.4 (NC), U6.5 (NC)
- new net: U6.19 (RESV), U6.21 (RESV), U6.22 (RESV)
- new net 12: J3.4 (Pin_4), U4.14 (IO12)
- new net 14: J3.3 (Pin_3), U4.13 (IO14)
- new net 27: J3.2 (Pin_2), U4.12 (IO27)
- new net 34: J3.1 (Pin_1), U4.6 (IO34)
- new net ADC_Batt: R16.2, R17.1, U4.7 (IO35)
- new net Buzz: R20.1, U4.29 (IO5)
- new net DTR: Q3.2 (E), R8.2, U5.13 (~{DTR})
- new net Down: C26.2, R22.1, SW5.1 (A), U4.11 (IO26)
- new net ENA: R19.2, U1.3 (EN), U2.3 (EN)
- new net IO0: C8.2, Q3.3 (C), R13.1, SW3.2 (B), U4.25 (IO0)
- new net Mode: C25.2, R21.1, SW4.1 (A), U4.10 (IO25)
- new net RTS: Q2.2 (E), R9.2, U5.14 (~{RTS})
- new net RX: D5.1 (K), U4.35 (TXD0/IO1), U5.3 (RXD)
- new net RX2: J5.2 (Pin_2), U4.27 (IO16)
- new net SCL: J4.3 (Pin_3), J6.3 (Pin_3), J7.2 (Pin_2), R15.2, U4.36 (IO22), U6.24 (SDA)
- new net SDA: J4.4 (Pin_4), J6.4 (Pin_4), J7.3 (Pin_3), R14.1, U4.33 (IO21), U6.23 (SCL)
- new net Select: C27.2, R23.1, SW6.1 (A), U4.8 (IO32)
- new net TX: D6.1 (K), U4.34 (RXD0/IO3), U5.2 (TXD)
- new net TX2: J5.3 (Pin_3), U4.28 (IO17)
- new net Up: C28.2, R24.1, SW7.1 (A), U4.9 (IO33)
- new net motor: Q4.1, U4.30 (IO18)
- no-connect marks 2 -> 23
Other:
- note added: "Batt Charging"
- note added: "Batt+ Charger"
- note added: "Control Switches"
- note added: "MPU6050"
- note added: "Sensors"
- note added: "SoC Module"
- note added: "TTL Converter"
- note added: "Utility Watch"
- note added: "motor"
- moved on the sheet: C13, C14, C15, C16

Commit message: updating PCB_watchV3
Parts:
- removed BZ1: Buzzer, Buzzer_Beeper:Buzzer_12x9.5RM7.6, symbol Device:Buzzer
- removed R20: 2.2E, Resistor_SMD:R_01005_0402Metric, symbol Device:R
- added D7: SS34, Capacitor_SMD:ss34_DO, symbol SS34:SS34
- added LS1: CMT-8530S-SMT, Capacitor_SMD:CUI_CMT-8530S-SMT, symbol CMT-8530S-SMT:CMT-8530S-SMT
- added Q5: BC847, Package_TO_SOT_SMD:SOT-23, symbol Transistor_BJT:BC847
- SW1, SW3: footprint Button_Switch_SMD:SW_Push_1P1T_NO_6x6mm_H9.5mm -> Button_Switch_SMD:SW_Tactile_SPST_NO_Straight_CK_PTS636Sx25SMTRLFS
Connections:
- net +3.3V: now also D7.C, LS1.P
- net Buzz: now also Q5.1 (B)
- net GND: now also Q5.2 (E)
- new net: D7.A, LS1.N, Q5.3 (C)
- no-connect marks 23 -> 28
Other:
- moved on the sheet: J3

Commit message: updating watchV3
Parts:
- removed C4, C5: 22pF, Capacitor_SMD:C_0402_1005Metric, symbol Device:C
- removed C6: 0.1uF, Capacitor_SMD:C_0402_1005Metric, symbol Device:C
- removed U5: CH340G, Package_SO:SOIC-16_3.9x9.9mm_P1.27mm, symbol Interface_USB:CH340G
- removed Y1: 12M, Crystal:Crystal_HC49-4H_Vertical, symbol Device:Crystal
- added U5: CP2102N-Axx-xQFN28, Package_DFN_QFN:QFN-28-1EP_5x5mm_P0.5mm_EP3.35x3.35mm, symbol Interface_USB:CP2102N-Axx-xQFN28
- SW4, SW5, SW6, SW7: footprint Button_Switch_SMD:SW_Push_1P1T_NO_6x6mm_H9.5mm -> Button_Switch_SMD:SW_Tactile_SPST_NO_Straight_CK_PTS636Sx25SMTRLFS
Connections:
- new net: U5.29 (GND), U5.3 (GND)
- no-connect marks 28 -> 37
Other:
- note removed: "TTL Converter"
- note removed: "Utility Watch"
- moved on the sheet: C10, C11, C12, C13, C14, C15, C16, C17, C18, C19, C2, C20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

Commit message: updating watch_V3
Parts:
- added C4, C5, C6: 0.1uF, Capacitor_SMD:C_0402_1005Metric, symbol Device:C
- added R20, R25, R26, R27, R29, R33, R34, R35, R36, R37, R38, R39: 0, Resistor_SMD:R_0402_1005Metric, symbol Device:R
- added R30, R31: 220E, Resistor_SMD:R_0402_1005Metric, symbol Device:R
- added R32: 4.7K, Resistor_SMD:R_0402_1005Metric, symbol Device:R
- D1: footprint Capacitor_SMD:ss34_DO -> Button_Switch_SMD:P25_DO-214AC_SMA
- D7: value SS34 -> 1N4148; footprint Capacitor_SMD:ss34_DO -> Diode_SMD:D_SOD-323
- J1: footprint Connector_USB:USB_C_Receptacle_HCTL_HC-TYPE-C-16P-01A -> Connector_USB:USB_C_Receptacle_GCT_USB4105-xx-A_16P_TopMnt_Horizontal
- R1, R10, R11, R12, R13, R14, R15, R16, R17, R18, R19, R2, R21, R22, R23, R24, R3, R4, R5, R6, R7, R8, R9: footprint Resistor_SMD:R_01005_0402Metric -> Resistor_SMD:R_0402_1005Metric
Connections:
- net +3.3V: now also R25.1, R26.1, R27.1, R29.1, R35.2, R36.1, R37.1, R39.1; no longer C21.1, C9.2, D7.C, J4.2 (Pin_2), J5.4 (Pin_4), J6.2 (Pin_2), LS1.P, Q4.3, U1.5 (VOUT), U2.5 (VOUT), U4.2 (VDD), U6.13 (VDD), U6.8 (VLOGIC)
- net +5V: now also R20.2, R38.1; no longer C3.2, D1.A, Q1.1 (G), R3.1, U3.4 (VCC)
- net D+: now also U5.4 (D+)
- net D-: now also U5.5 (D-)
- net DTR: now also U5.28 (~{DTR})
- net GND: now also J3.1 (Pin_1), U5.29 (GND), U5.3 (GND), C4.2, C5.1, C6.1
- net RTS: now also U5.24 (~{RTS})
- net RX: now also R30.2
- net SCL: now also U6.23 (SCL); no longer U6.24 (SDA)
- net SDA: now also U6.24 (SDA); no longer U6.23 (SCL)
- net TX: now also R31.1
- net VBUS: now also U5.7 (VREGIN), C5.2, C6.2, R33.1, R34.1; no longer C2.2, D1.C, Q1.3 (D)
- net at U5.25 (RXD): now also R30.1
- net at U5.26 (TXD): now also R31.2
- net at U5.6 (VDD): now also C4.1, R32.1
- net at U5.8 (VBUS): now also R33.2
- net at U5.9 (~{RST}): now also R32.2
- net 34: no longer names the net of U4.6 (IO34)
- net 34: no longer J3.1 (Pin_1)
- new net: R38.2, U3.4 (VCC)
- new net: J5.4 (Pin_4), R26.2
- new net: R25.2, U1.5 (VOUT), U2.5 (VOUT)
- new net: J4.2 (Pin_2), R37.2
- new net: C9.2, R35.1, U4.2 (VDD)
- new net: C3.2, D1.A, Q1.1 (G), R20.1, R3.1
- new net: D7.C, LS1.P, R29.2
- new net: C2.2, D1.C, Q1.3 (D), R34.2
- new net: Q4.3, R27.2
- new net: C21.1, R36.2, U6.13 (VDD), U6.8 (VLOGIC)
- new net: J6.2 (Pin_2), R39.2
- no-connect marks 37 -> 42
Other:
- note added: "ADC_V"
- note added: "Charger"
- note added: "Power Switch"
- note added: "SoC"
- note added: "USB-UART"
- note added: "Utility Watch"
- note removed: "Batt Charging"
- note removed: "Batt+ Charger"
- note removed: "On/Off Switch"
- note removed: "SoC Module"
- moved on the sheet: C1, C10, C11, C12, C13, C14, C15, C16, C17, C18, C19, C2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

Commit message: remote_v3
Parts:
- added J8: ICSP, Button_Switch_SMD:solder_pad_4, symbol Connector:Conn_01x04_Pin
Connections:
- net +5V: now also J8.4 (Pin_4)
- net GND: now also J8.1 (Pin_1)
- net RX: now also J8.3 (Pin_3)
- net TX: now also J8.2 (Pin_2)
Changed lines of the file:
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@@
     (effects (font (size 1 1)) (justify left bottom))
   )
+  (label "TX" (at 181.61 58.42 180) (fields_autoplaced)
+    (effects (font (size 1 1)) (justify right bottom))
+  )
   (label "RTS" (at 69.85 114.935 180) (fields_autoplaced)
     (effects (font (size 1 1)) (justify right bottom))
@@
     (effects (font (size 1 1)) (justify right bottom))
   )
+  (label "RX" (at 181.61 55.88 180) (fields_autoplaced)
+    (effects (font (size 1 1)) (justify right bottom))
+  )
   (label "ADC_Batt" (at 111.76 112.395 270) (fields_autoplaced)
     (effects (font (size 1 1)) (justify right bottom))
@@
     )
   )
+  (symbol (lib_id "power:+5V") (at 181.61 53.34 0) (unit 1)
+    (in_bom yes) (on_board yes) (dnp no)
+    (property "Reference" "#PWR045" (at 181.61 57.15 0)
+      (effects (font (size 1.27 1.27)) hide)
+    )
+    (property "Value" "+5V" (at 181.61 49.53 0)
+      (effects (font (size 1 1)))
+    )
+    (property "Footprint" "" (at 181.61 53.34 0)
+      (effects (font (size 1.27 1.27)) hide)
+    )
+    (property "Datasheet" "" (at 181.61 53.34 0)
+      (effects (font (size 1.27 1.27)) hide)
+    )
+    (pin "1")
+    (instances
+      (project "Watch_v3"
+        (path "/a181cade-ee2d-4579-b71a-76068187d0cf"
+          (reference "#PWR045") (unit 1)
+        )
+      )
+    )
+  )
   (symbol (lib_id "SS34:SS34") (at 65.405 37.465 0) (unit 1)
     (in_bom yes) (on_board yes) (dnp no)
@@
     )
   )
+  (symbol (lib_id "power:GND") (at 181.61 60.96 270) (unit 1)
+    (in_bom yes) (on_board yes) (dnp no)
+    (property "Reference" "#PWR070" (at 175.26 60.96 0)
+      (effects (font (size 1.27 1.27)) hide)
+    )
+    (property "Value" "GND" (at 178.435 60.96 0)
+      (effects (font (size 1 1)))
+    )
+    (property "Footprint" "" (at 181.61 60.96 0)
+      (effects (font (size 1.27 1.27)) hide)
+    )
+    (property "Datasheet" "" (at 181.61 60.96 0)
+      (effects (font (size 1.27 1.27)) hide)
+    )
+    (pin "1")
+    (instances
+      (project "Watch_v3"
+        (path "/a181cade-ee2d-4579-b71a-76068187d0cf"
+          (reference "#PWR070") (unit 1)
+        )
+      )
+    )
+  )
   (symbol (lib_id "Device:R") (at 107.315 112.395 90) (unit 1)
     (in_bom yes) (on_board yes) (dnp no)
@@
         )
       )
+    )
+  )
+  (symbol (lib_id "Connector:Conn_01x04_Pin") (at 186.69 58.42 180) (unit 1)
+    (in_bom yes) (on_board yes) (dnp no)
+    (property "Reference" "J8" (at 186.69 57.15 0)
+      (effects (font (size 1 1)) (justify right))
+    )
+    (property "Value" "ICSP" (at 182.245 62.23 0)
+      (effects (font (size 1 1)) (justify right))
+    )
+    (property "Footprint" "Button_Switch_SMD:solder_pad_4" (at 186.69 58.42 0)
+      (effects (font (size 1.27 1.27)) hide)
+    )
+    (property "Datasheet" "~" (at 186.69 58.42 0)
+      (effects (font (size 1.27 1.27)) hide)
+    )
+    (pin "3")
+    (pin "4")
+    (pin "1")
+    (pin "2")
+    (instances
+      (project "Watch_v3"
+        (path "/a181cade-ee2d-4579-b71a-76068187d0cf"
+          (reference "J8") (unit 1)
+        )
+      )
