File: PCB/Watch_V3/Watch_v3.kicad_sch (KiCad schematic)
At the start: 100 parts, among them J1 USB_C_Receptacle_USB2.0_16P, J2 Screw_Terminal, J3 Peripheral, J4 OLED, J5 BN220, J6 Peripheral, J7 MAX30102, J8 ICSP, M1 Motor_DC, Q1 AO3401A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

Commit message: update watch_v3
Parts:
- SW4: value Select -> Mode
- SW5: value Mode -> Down
- SW6: value Up -> Select
- SW7: value Down -> Up
Changed lines of the file:
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@@
       (effects (font (size 1 1)) (justify right))
     )
-    (property "Value" "Up" (at 46.355 179.07 0)
+    (property "Value" "Select" (at 46.355 179.07 0)
       (effects (font (size 1 1)) (justify right))
     )
@@
       (effects (font (size 1 1)) (justify right))
     )
-    (property "Value" "Down" (at 60.96 178.435 0)
+    (property "Value" "Up" (at 60.96 180.34 0)
       (effects (font (size 1 1)) (justify right))
     )
@@
       (effects (font (size 1 1)) (justify right))
     )
-    (property "Value" "Mode" (at 33.655 178.435 0)
+    (property "Value" "Down" (at 33.655 178.435 0)
       (effects (font (size 1 1)) (justify right))
     )
@@
       (effects (font (size 1 1)) (justify right))
     )
-    (property "Value" "Select" (at 18.415 178.435 0)
-      (effects (font (size 1 1)) (justify right))
-    )
+    (property "Value" "Mode" (at 18.415 178.435 0)
+      (effects (font (size 1 1)) (justify right))
+    )
