File: PCB/Watch_V3/Watch_v3.kicad_sch (KiCad schematic)
At the start: 80 parts, among them J1 USB_C_Receptacle_USB2.0_16P, J2 Screw_Terminal, J3 Peripheral, J4 OLED, J5 BN220, J7 MAX30102, J8 Conn_01x07_Pin, M1 Motor_DC, Q1 AO3401A, Q4 SI2302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

Commit message: update watch_v3
Parts:
- removed J3: Peripheral, Button_Switch_SMD:solder_pad_4, symbol Connector:Conn_01x04_Pin
- U3: footprint TP4056:SOP127P600X175-9N -> Package_SO:HSOP-8-1EP_3.9x4.9mm_P1.27mm_EP2.3x2.3mm
- U6: footprint Button_Switch_SMD:QFN50P400X400X95-24N -> Package_DFN_QFN:QFN-24-1EP_3x3mm_P0.4mm_EP1.75x1.6mm
Connections:
- no-connect marks 30 -> 32
Changed lines of the file:
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@@
   (no_connect (at 235.585 64.77))
   (no_connect (at 158.75 20.32))
+  (no_connect (at 152.4 104.14))
+  (no_connect (at 152.4 109.22))
   (no_connect (at 266.065 57.15))
   (no_connect (at 235.585 69.85))
@@
     (effects (font (size 1 1)) (justify right bottom))
   )
-  (label "27" (at 170.18 58.42 180) (fields_autoplaced)
-    (effects (font (size 1.27 1.27)) (justify right bottom))
-  )
   (label "ADC_Batt" (at 266.065 92.71 0) (fields_autoplaced)
     (effects (font (size 1 1)) (justify left bottom))
   )
-  (label "14" (at 170.18 55.88 180) (fields_autoplaced)
-    (effects (font (size 1.27 1.27)) (justify right bottom))
-  )
   (label "motor" (at 266.065 64.77 0) (fields_autoplaced)
     (effects (font (size 1 1)) (justify left bottom))
@@
     (effects (font (size 1 1)) (justify right bottom))
   )
-  (label "12" (at 170.18 53.34 180) (fields_autoplaced)
-    (effects (font (size 1.27 1.27)) (justify right bottom))
-  )
   (label "Down" (at 39.37 100.33 270) (fields_autoplaced)
     (effects (font (size 1.27 1.27)) (justify right bottom))
@@
       (effects (font (size 1 1)))
     )
-    (property "Footprint" "TP4056:SOP127P600X175-9N" (at 241.3 139.065 0)
+    (property "Footprint" "Package_SO:HSOP-8-1EP_3.9x4.9mm_P1.27mm_EP2.3x2.3mm" (at 241.3 139.065 0)
       (effects (font (size 1.27 1.27)) (justify bottom) hide)
     )
@@
     )
   )
-  (symbol (lib_id "Connector:Conn_01x04_Pin") (at 175.26 58.42 180) (unit 1)
-    (in_bom yes) (on_board yes) (dnp no)
-    (property "Reference" "J3" (at 175.26 57.15 0)
-      (effects (font (size 1 1)) (justify right))
-    )
-    (property "Value" "Peripheral" (at 169.545 62.23 0)
-      (effects (font (size 1 1)) (justify right))
-    )
-    (property "Footprint" "Button_Switch_SMD:solder_pad_4" (at 175.26 58.42 0)
-      (effects (font (size 1.27 1.27)) hide)
-    )
-    (property "Datasheet" "~" (at 175.26 58.42 0)
-      (effects (font (size 1.27 1.27)) hide)
-    )
-    (pin "3")
-    (pin "4")
-    (pin "1")
-    (pin "2")
-    (instances
-      (project "Watch_v3"
-        (path "/a181cade-ee2d-4579-b71a-76068187d0cf"
-          (reference "J3") (unit 1)
-        )
-      )
-    )
-  )
   (symbol (lib_id "power:+5V") (at 271.78 135.255 0) (unit 1)
     (in_bom yes) (on_board yes) (dnp no)
@@
     )
   )
-  (symbol (lib_id "power:GND") (at 170.18 60.96 270) (unit 1)
-    (in_bom yes) (on_board yes) (dnp no)
-    (property "Reference" "#PWR024" (at 163.83 60.96 0)
-      (effects (font (size 1.27 1.27)) hide)
-    )
-    (property "Value" "GND" (at 166.37 60.96 0)
-      (effects (font (size 1 1)))
-    )
-    (property "Footprint" "" (at 170.18 60.96 0)
-      (effects (font (size 1.27 1.27)) hide)
-    )
-    (property "Datasheet" "" (at 170.18 60.96 0)
-      (effects (font (size 1.27 1.27)) hide)
-    )
-    (pin "1")
-    (instances
-      (project "Watch_v3"
-        (path "/a181cade-ee2d-4579-b71a-76068187d0cf"
-          (reference "#PWR024") (unit 1)
-        )
-      )
-    )
-  )
   (symbol (lib_id "power:GND") (at 276.86 41.91 0) (unit 1)
     (in_bom yes) (on_board yes) (dnp no)
@@
       (effects (font (size 1.27 1.27)))
     )
-    (property "Footprint" "Button_Switch_SMD:QFN50P400X400X95-24N" (at 170.18 101.6 0)
+    (property "Footprint" "Package_DFN_QFN:QFN-24-1EP_3x3mm_P0.4mm_EP1.75x1.6mm" (at 170.18 101.6 0)
       (effects (font (size 1.27 1.27)) (justify bottom) hide)
     )

Commit message: updating PCBs
Parts:
- R14: value 1K -> 10K
Other:
- moved on the sheet: C17, C18, C19, C20, D7, J4, J5, J7, LS1, Q5, R29

Commit message: updating PCB design
Connections:
- net VBUS: now also C2.2
- net at D1.C, Q1.3 (D), R34.2: no longer C2.2
Changed lines of the file:
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@@
+    (stroke (width 0) (type default))
+  )
+  (wire (pts (xy 78.105 41.275) (xy 78.105 37.465))
     (stroke (width 0) (type default))
   )
@@
     (stroke (width 0) (type default))
   )
-  (wire (pts (xy 70.485 37.465) (xy 70.485 41.275))
-    (stroke (width 0) (type default))
-  )
   (wire (pts (xy 44.45 100.33) (xy 44.45 97.79))
     (stroke (width 0) (type default))
@@
     (stroke (width 0) (type default))
   )
+  (wire (pts (xy 71.755 41.275) (xy 78.105 41.275))
+    (stroke (width 0) (type default))
+  )
   (wire (pts (xy 106.045 37.465) (xy 111.76 37.465))
     (stroke (width 0) (type default))
@@
     (stroke (width 0) (type default))
   )
-  (wire (pts (xy 70.485 41.275) (xy 71.755 41.275))
-    (stroke (width 0) (type default))
-  )
