File: PCB/Remote_V2/UART.kicad_sch (KiCad schematic)
At the start: 48 parts, among them Q11 BC817, Q12 BC817, Q13 BC817, Q14 BC817, Q6 BC817, Q7 BC817, U18 CP2102N-Axx-xQFN28, U19 CP2102N-Axx-xQFN28, U20 CP2102N-Axx-xQFN28

Commit message: remote_v2 update
Other:
- note added: "CP2102 USB-UART"
- note added: "H"
- company: (none) -> Dharma Bot KRS
- title: (none) -> UART_Utility_Remote
Changed lines of the file:
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@@
 (kicad_sch (version 20230121) (generator eeschema)
   (paper "A4")
+  (title_block
+    (title "UART_Utility_Remote")
+    (date "2024-11-28")
+    (rev "V2")
+    (company "Dharma Bot KRS")
+  )
   (junction (at 60.325 66.675) (diameter 0) (color 0 0 0 0)
   )
@@
     (stroke (width 0) (type default))
   )
+  (rectangle (start 39.37 144.145) (end 87.63 174.625)
+    (stroke (width 0.3) (type dash) (color 255 16 12 1))
+    (fill (type none))
+  )
   (rectangle (start 39.37 57.15) (end 104.14 140.335)
     (stroke (width 0.3) (type dash) (color 255 16 12 1))
@@
     (effects (font (size 2 2) (thickness 0.4) bold) (justify left bottom))
   )
+  (text "H\n" (at 83.185 147.955 0)
+    (effects (font (size 2 2) (thickness 0.4) bold) (justify left bottom))
+  )
+  (text "CP2102 USB-UART\n\n" (at 168.91 53.34 0)
+    (effects (font (size 6 6) (thickness 1.6) bold (color 253 61 255 1)) (justify left bottom))
+  )
   (text "USB-UART" (at 87.63 61.595 0)
     (effects (font (size 2 2) (thickness 0.4) bold) (justify left bottom))
@@
     (effects (font (size 1 1)) (justify left bottom))
   )
+  (label "TX3" (at 55.88 168.91 0) (fields_autoplaced)
+    (effects (font (size 1 1)) (justify left bottom))
+  )
+  (label "D1-" (at 57.15 153.035 0) (fields_autoplaced)
+    (effects (font (size 1.27 1.27)) (justify left bottom))
+  )
+  (label "EN1" (at 53.975 161.29 180) (fields_autoplaced)
+    (effects (font (size 1 1)) (justify right bottom))
+  )
+  (label "IO01" (at 57.15 161.29 0) (fields_autoplaced)
+    (effects (font (size 1 1)) (justify left bottom))
+  )
+  (label "D3-" (at 81.28 153.035 0) (fields_autoplaced)
+    (effects (font (size 1.27 1.27)) (justify left bottom))
+  )
   (label "D1+" (at 47.625 90.805 180) (fields_autoplaced)
     (effects (font (size 1.27 1.27)) (justify right bottom))
@@
     (effects (font (size 1 1)) (justify left bottom))
   )
+  (label "D2-" (at 68.58 153.035 0) (fields_autoplaced)
+    (effects (font (size 1.27 1.27)) (justify left bottom))
+  )
   (label "DTR2" (at 156.845 82.55 180) (fields_autoplaced)
     (effects (font (size 1 1)) (justify right bottom))
   )
+  (label "D3+" (at 74.295 153.035 0) (fields_autoplaced)
+    (effects (font (size 1.27 1.27)) (justify left bottom))
+  )
+  (label "D2+" (at 62.23 153.035 0) (fields_autoplaced)
+    (effects (font (size 1.27 1.27)) (justify left bottom))
+  )
+  (label "TX2" (at 62.865 161.29 0) (fields_autoplaced)
+    (effects (font (size 1 1)) (justify left bottom))
+  )
   (label "RTS2" (at 172.085 89.535 180) (fields_autoplaced)
     (effects (font (size 1 1)) (justify right bottom))
@@
     (effects (font (size 1.27 1.27)) (justify right bottom))
   )
+  (label "IO02" (at 79.375 161.29 0) (fields_autoplaced)
+    (effects (font (size 1 1)) (justify left bottom))
+  )
   (label "D3+" (at 199.39 90.805 180) (fields_autoplaced)
     (effects (font (size 1.27 1.27)) (justify right bottom))
@@
     (effects (font (size 1 1)) (justify left bottom))
   )
+  (label "IO03" (at 71.12 168.91 0) (fields_autoplaced)
+    (effects (font (size 1 1)) (justify left bottom))
+  )
   (label "D2-" (at 125.095 88.265 180) (fields_autoplaced)
     (effects (font (size 1.27 1.27)) (justify right bottom))
@@
     (effects (font (size 1 1)) (justify right bottom))
   )
+  (label "RX3" (at 60.96 168.91 0) (fields_autoplaced)
+    (effects (font (size 1 1)) (justify left bottom))
+  )
   (label "RX3" (at 232.41 74.93 0) (fields_autoplaced)
     (effects (font (size 1 1)) (justify left bottom))
@@
     (effects (font (size 1 1)) (justify right bottom))
   )
+  (label "D1+" (at 51.435 153.035 0) (fields_autoplaced)
+    (effects (font (size 1.27 1.27)) (justify left bottom))
+  )
   (label "RTS1" (at 94.615 89.535 180) (fields_autoplaced)
     (effects (font (size 1 1)) (justify right bottom))
@@
     (effects (font (size 1 1)) (justify left bottom))
   )
+  (label "EN2" (at 75.565 161.29 180) (fields_autoplaced)
+    (effects (font (size 1 1)) (justify right bottom))
+  )
   (label "EN2" (at 172.085 79.375 180) (fields_autoplaced)
     (effects (font (size 1 1)) (justify right bottom))
@@
     (effects (font (size 1 1)) (justify left bottom))
   )
+  (label "TX1" (at 41.91 161.29 0) (fields_autoplaced)
+    (effects (font (size 1 1)) (justify left bottom))
+  )
   (label "RTS3" (at 231.14 97.79 180) (fields_autoplaced)
     (effects (font (size 1 1)) (justify right bottom))
@@
     (effects (font (size 1 1)) (justify right bottom))
   )
+  (label "RX2" (at 67.945 161.29 0) (fields_autoplaced)
+    (effects (font (size 1 1)) (justify left bottom))
+  )
+  (label "EN3" (at 67.945 168.91 180) (fields_autoplaced)
+    (effects (font (size 1 1)) (justify right bottom))
+  )
+  (label "RX1" (at 46.355 161.29 0) (fields_autoplaced)
+    (effects (font (size 1 1)) (justify left bottom))
+  )
   (label "RX1" (at 80.645 74.93 0) (fields_autoplaced)
     (effects (font (size 1 1)) (justify left bottom))
@@
   (label "RX2" (at 158.115 74.93 0) (fields_autoplaced)
     (effects (font (size 1 1)) (justify left bottom))
+  )
+  (hierarchical_label "TX3" (shape input) (at 55.88 168.91 270) (fields_autoplaced)
+    (effects (font (size 1 1)) (justify right))
+  )
+  (hierarchical_label "D1-" (shape input) (at 57.15 153.035 270) (fields_autoplaced)
+    (effects (font (size 1 1)) (justify right))
+  )
+  (hierarchical_label "EN2" (shape input) (at 75.565 161.29 270) (fields_autoplaced)
+    (effects (font (size 1 1)) (justify right))
+  )
+  (hierarchical_label "D2-" (shape input) (at 68.58 153.035 270) (fields_autoplaced)
+    (effects (font (size 1 1)) (justify right))
+  )
+  (hierarchical_label "TX1" (shape input) (at 41.91 161.29 270) (fields_autoplaced)
+    (effects (font (size 1 1)) (justify right))
+  )
+  (hierarchical_label "IO03" (shape input) (at 71.12 168.91 270) (fields_autoplaced)
+    (effects (font (size 1 1)) (justify right))
+  )
+  (hierarchical_label "VBUS" (shape input) (at 46.99 153.67 270) (fields_autoplaced)
+    (effects (font (size 1 1)) (justify right))
+  )
+  (hierarchical_label "D2+" (shape input) (at 62.23 153.035 270) (fields_autoplaced)
+    (effects (font (size 1 1)) (justify right))
+  )
+  (hierarchical_label "D1+" (shape input) (at 51.435 153.035 270) (fields_autoplaced)
+    (effects (font (size 1 1)) (justify right))
+  )
+  (hierarchical_label "EN3" (shape input) (at 67.945 168.91 270) (fields_autoplaced)
+    (effects (font (size 1 1)) (justify right))
+  )
+  (hierarchical_label "D3-" (shape input) (at 81.28 153.035 270) (fields_autoplaced)
+    (effects (font (size 1 1)) (justify right))
+  )
+  (hierarchical_label "TX2" (shape input) (at 62.865 161.29 270) (fields_autoplaced)
+    (effects (font (size 1 1)) (justify right))
+  )
+  (hierarchical_label "RX2" (shape input) (at 67.945 161.29 270) (fields_autoplaced)
+    (effects (font (size 1 1)) (justify right))
+  )
+  (hierarchical_label "D3+" (shape input) (at 74.295 153.035 270) (fields_autoplaced)
+    (effects (font (size 1 1)) (justify right))
+  )
+  (hierarchical_label "EN1" (shape input) (at 53.975 161.29 270) (fields_autoplaced)
+    (effects (font (size 1 1)) (justify right))
+  )
+  (hierarchical_label "RX1" (shape input) (at 46.355 161.29 270) (fields_autoplaced)
+    (effects (font (size 1 1)) (justify right))
+  )
+  (hierarchical_label "GND" (shape input) (at 42.545 153.67 270) (fields_autoplaced)
+    (effects (font (size 1 1)) (justify right))
+  )
+  (hierarchical_label "RX3" (shape input) (at 60.96 168.91 270) (fields_autoplaced)
+    (effects (font (size 1 1)) (justify right))
+  )
+  (hierarchical_label "IO01" (shape input) (at 57.15 161.29 270) (fields_autoplaced)
+    (effects (font (size 1 1)) (justify right))
+  )
+  (hierarchical_label "IO02" (shape input) (at 79.375 161.29 270) (fields_autoplaced)
+    (effects (font (size 1 1)) (justify right))
   )
   (symbol (lib_id "Device:R") (at 51.435 66.675 270) (unit 1)
@@
         (path "/06398ea7-2a88-46d2-a66c-c169b1a4e04e/4a30931c-a518-4c65-958d-7215ff99da7b"
           (reference "#PWR0141") (unit 1)
+        )
+      )
+    )
+  )
+  (symbol (lib_id "power:VBUS") (at 46.99 153.67 0) (unit 1)
+    (in_bom yes) (on_board yes) (dnp no)
+    (property "Reference" "#PWR0213" (at 46.99 157.48 0)
+      (effects (font (size 1.27 1.27)) hide)
+    )
+    (property "Value" "VBUS" (at 46.99 150.495 0)
+      (effects (font (size 1 1)))
+    )
+    (property "Footprint" "" (at 46.99 153.67 0)
+      (effects (font (size 1.27 1.27)) hide)
+    )
+    (property "Datasheet" "" (at 46.99 153.67 0)
+      (effects (font (size 1.27 1.27)) hide)
+    )
+    (pin "1")
+    (instances
+      (project "remote_v2"
+        (path "/06398ea7-2a88-46d2-a66c-c169b1a4e04e/4a30931c-a518-4c65-958d-7215ff99da7b"
+          (reference "#PWR0213") (unit 1)
         )
       )
@@
         )
       )
+    )
+  )
+  (symbol (lib_id "power:GND") (at 42.545 153.67 180) (unit 1)
+    (in_bom yes) (on_board yes) (dnp no)
+    (property "Reference" "#PWR0214" (at 42.545 147.32 0)
+      (effects (font (size 1.27 1.27)) hide)
+    )
+    (property "Value" "GND" (at 42.545 149.86 0)
+      (effects (font (size 1 1)))
+    )
+    (property "Footprint" "" (at 42.545 153.67 0)
+      (effects (font (size 1.27 1.27)) hide)
+    )
+    (property "Datasheet" "" (at 42.545 153.67 0)
+      (effects (font (size 1.27 1.27)) hide)
+    )
+    (pin "1")
+    (instances
+      (project "remote_v2"
+        (path "/06398ea7-2a88-46d2-a66c-c169b1a4e04e/4a30931c-a518-4c65-958d-7215ff99da7b"
+          (reference "#PWR0214") (unit 1)
+        )
+      )
