File: PCB/Remote_V2/buck.kicad_sch (KiCad schematic)
At the start: 35 parts, among them J17 XT60-M

Commit message: updating watch_v3
Parts:
- removed C62, C70, C72, C82, C83, C85, C86, C88: 100uF, Battery:CAPAE830X1000N, symbol UWT1V101MCL1GS:UWT1V101MCL1GS
- J17: footprint Button_Switch_SMD:AMASS_XT60-M -> Battery:AMASS_XT60PW-M
Connections:
- net GND: now also J17.2 (NEG); no longer J17.N (NEG)
- net Vin: now also J17.1 (POS); no longer J17.P (POS)
Other:
- moved on the sheet: C26, C29, C35, C60, C61, C71, C84, C87
