File: PCB/Remote_V2/buck.kicad_sch (KiCad schematic)
At the start: 13 parts, among them J17 XT60-M

Commit message: updating PCBs
Parts:
- removed U8: ~, Audio_Module:5v_usbbuck, symbol Triac_Thyristor:5vusbbuck
Other:
- moved on the sheet: C35, C59, C60, C61, C71
