File: PCB/Remote_V2/remote_v2.kicad_pcb (KiCad board)
At the start: 2 copper layers, 161 parts, among them J1 USB_C_Receptacle_USB2.0_16P, J5 USB_C_Receptacle_USB2.0_16P, J6 USB_C_Receptacle_USB2.0_16P, Q1 AO3401A, Q11 BC817, Q12 BC817, Q13 BC817, Q14 BC817, Q2 AO3401A, Q3 AO3401A, Q6 BC817, Q7 BC817, SW1 SW_DPST_x2, SW10 SW_DPST_x2, SW11 SW_DPST_x2, SW2 SW_DPST_x2, SW3 SW_DPST_x2, SW4 SW_DPST_x2, SW5 SW_DPST_x2, SW6 SW_DPST_x2, U1 AP2112K-3.3, U10 ESP32-WROOM-32D, U16 AP2112K-3.3, U18 CP2102N-Axx-xQFN28, U19 CP2102N-Axx-xQFN28, U20 CP2102N-Axx-xQFN28, U3 AP2112K-3.3, U4 AP2112K-3.3, U5 AP2112K-3.3, U6 ESP32-WROOM-32D, U7 AP2112K-3.3, U8 ESP32-WROOM-32D, U9 ESP32-WROOM-32D

Commit message: remote_v2 update
Parts:
- removed SW10, SW11: SW_DPST_x2, Button_Switch_SMD:SW_Tactile_SPST_NO_Straight_CK_PTS636Sx25SMTRLFS
- added C36: 0.1uF, Capacitor_SMD:C_0402_1005Metric, F.Cu at (532.3, 86.2)
- added C37: 0.1uF, Capacitor_SMD:C_0402_1005Metric, F.Cu at (532.3, 88.2)
- added C38: 0.1uF, Capacitor_SMD:C_0402_1005Metric, F.Cu at (532.3, 90.2)
- added C39: 0.1uF, Capacitor_SMD:C_0402_1005Metric, F.Cu at (532.3, 92.1)
- added C40: 0.1uF, Capacitor_SMD:C_0402_1005Metric, F.Cu at (535.1, 80.3)
- added C41: 0.1uF, Capacitor_SMD:C_0402_1005Metric, F.Cu at (535.1, 82.3)
- added C42: 0.1uF, Capacitor_SMD:C_0402_1005Metric, F.Cu at (535.1, 84.3)
- added C43: 0.1uF, Capacitor_SMD:C_0402_1005Metric, F.Cu at (535.1, 86.2)
- added C44: 0.1uF, Capacitor_SMD:C_0402_1005Metric, F.Cu at (535.1, 88.2)
- added C45: 0.1uF, Capacitor_SMD:C_0402_1005Metric, F.Cu at (535.1, 90.2)
- added C46: 0.1uF, Capacitor_SMD:C_0402_1005Metric, F.Cu at (535.1, 92.1)
- added C47: 100uF, Capacitor_SMD:C_0402_1005Metric, F.Cu at (538.0, 80.3)
- added C48: 100uF, Capacitor_SMD:C_0402_1005Metric, F.Cu at (538.0, 82.3)
- added C49: 0.1uF, Capacitor_SMD:C_0402_1005Metric, F.Cu at (538.0, 84.3)
- added C50: 0.1uF, Capacitor_SMD:C_0402_1005Metric, F.Cu at (538.0, 86.2)
- added C51: 2.2nF, Capacitor_SMD:C_0402_1005Metric, F.Cu at (538.0, 88.2)
- added C52: 0.1uF, Capacitor_SMD:C_0402_1005Metric, F.Cu at (538.0, 90.2)
- added C53: 0.1uF, Capacitor_SMD:C_0402_1005Metric, F.Cu at (538.0, 92.1)
- added C54: 100uF, Battery:CAPAE830X1000N, F.Cu at (488.8, 74.6)
- added C55: 100uF, Battery:CAPAE830X1000N, F.Cu at (488.8, 84.5)
- added C56: 100uF, Battery:CAPAE830X1000N, F.Cu at (488.8, 94.3)
- added C57: 100uF, Battery:CAPAE830X1000N, F.Cu at (488.8, 104.2)
- added C58: 100uF, Battery:CAPAE830X1000N, F.Cu at (539.6, 174.0)
- added C59: 100uF, Battery:CAPAE830X1000N, F.Cu at (539.6, 183.8)
- added C60: 100uF, Battery:CAPAE830X1000N, F.Cu at (539.6, 193.7)
- added C61: 100uF, Battery:CAPAE830X1000N, F.Cu at (539.6, 203.5)
- added C62: 100uF, Battery:CAPAE830X1000N, F.Cu at (539.6, 213.4)
- added C70: 100uF, Battery:CAPAE830X1000N, F.Cu at (553.4, 154.3)
- added C71: 100uF, Battery:CAPAE830X1000N, F.Cu at (553.4, 164.1)
- added C72: 100uF, Battery:CAPAE830X1000N, F.Cu at (553.4, 174.0)
- added C82: 100uF, Battery:CAPAE830X1000N, F.Cu at (553.4, 183.8)
- added C83: 100uF, Battery:CAPAE830X1000N, F.Cu at (553.4, 193.7)
- added C84: 100uF, Battery:CAPAE830X1000N, F.Cu at (553.4, 203.5)
- added C85: 100uF, Battery:CAPAE830X1000N, F.Cu at (553.4, 213.4)
- added C86: 100uF, Battery:CAPAE830X1000N, F.Cu at (567.1, 154.3)
- added C87: 100uF, Battery:CAPAE830X1000N, F.Cu at (567.1, 164.1)
- added C88: 100uF, Battery:CAPAE830X1000N, F.Cu at (434.6, 54.6)
- added C89: 0.1uF, Capacitor_SMD:C_0402_1005Metric, F.Cu at (567.1, 174.0)
- added C90: 0.1uF, Capacitor_SMD:C_0402_1005Metric, F.Cu at (434.6, 56.5)
- added C91: 0.1uF, Capacitor_SMD:C_0402_1005Metric, F.Cu at (434.6, 58.5)
- added C92: 0.1uF, Capacitor_SMD:C_0402_1005Metric, F.Cu at (437.5, 54.6)
- added C93: 0.1uF, Capacitor_SMD:C_0402_1005Metric, F.Cu at (437.5, 56.5)
- added C94: 0.1uF, Capacitor_SMD:C_0402_1005Metric, F.Cu at (437.5, 58.5)
- added C95: 0.1uF, Capacitor_SMD:C_0402_1005Metric, F.Cu at (440.4, 54.6)
- added C96: 0.1uF, Capacitor_SMD:C_0402_1005Metric, F.Cu at (440.4, 56.5)
- added C97: 0.1uF, Capacitor_SMD:C_0402_1005Metric, F.Cu at (440.4, 58.5)
- added D11: 1N4148, Diode_SMD:D_SOD-323, F.Cu at (538.2, 102.6)
- added D12: 1N4148, Diode_SMD:D_SOD-323, F.Cu at (538.2, 105.6)
- added D13: LED, LED_SMD:LED_0402_1005Metric, F.Cu at (516.3, 104.5)
- added D14: LED, LED_SMD:LED_0402_1005Metric, F.Cu at (516.3, 106.5)
- added D7: 1N4148, Diode_SMD:D_SOD-323, F.Cu at (538.2, 96.7)
- added D8: 1N4148, Diode_SMD:D_SOD-323, F.Cu at (538.2, 99.7)
- added J10: Yaxis J1, Battery:smd_pad_10, F.Cu at (506.6, 89.7)
- added J11: Yaxis J2, Battery:smd_pad_10, F.Cu at (506.6, 93.8)
- added J12: Yaxis J3, Battery:smd_pad_10, F.Cu at (506.6, 98.0)
- added J13: Yaxis J4, Battery:smd_pad_10, F.Cu at (506.6, 102.1)
- added J14: ICSP1, Button_Switch_SMD:solder_pad_4, F.Cu at (499.4, 73.7)
- added J15: ICSP2, Button_Switch_SMD:solder_pad_4, F.Cu at (499.4, 78.5)
- added J16: ICSP3, Button_Switch_SMD:solder_pad_4, F.Cu at (499.4, 83.3)
- added J17: XT60-M, Button_Switch_SMD:AMASS_XT60-M, F.Cu at (455.8, 195.5)
- added J18: Peri Soc 1, Button_Switch_SMD:solder_pad_4, F.Cu at (499.4, 88.1)
- added J19: Peri Soc 2, Button_Switch_SMD:solder_pad_4, F.Cu at (499.4, 92.9)
- added J2: ADS1115 A1, Connector_PinHeader_2.54mm:PinHeader_1x10_P2.54mm_Vertical, F.Cu at (512.2, 72.0)
- added J20: Peri Soc 3, Button_Switch_SMD:solder_pad_4, F.Cu at (499.4, 97.7)
- added J21: UART Soc 1, Button_Switch_SMD:solder_pad_4, F.Cu at (499.4, 102.5)
- added J22: UART Soc 2, Button_Switch_SMD:solder_pad_4, F.Cu at (499.4, 107.3)
- added J23: UART Soc 3, Button_Switch_SMD:solder_pad_4, F.Cu at (499.4, 112.1)
- added J24: 5V, Button_Switch_SMD:solder_motor, F.Cu at (512.3, 107.2)
- added J25: XT60-M, Button_Switch_SMD:AMASS_XT60-M, F.Cu at (529.3, 74.5)
- added J26: UART RASP, Button_Switch_SMD:solder_pad_4, F.Cu at (356.4, 71.1)
- added J27: RASP Peripheral, Connector_PinHeader_2.54mm:PinHeader_1x10_P2.54mm_Vertical, F.Cu at (350.0, 69.3)
- added J3: ADS1115 A2, Connector_PinHeader_2.54mm:PinHeader_1x10_P2.54mm_Vertical, F.Cu at (516.9, 72.0)
- added J4: Xaxis J1, Battery:smd_pad_10, F.Cu at (506.6, 73.1)
- added J7: Xaxis J2, Battery:smd_pad_10, F.Cu at (506.6, 77.2)
- added J8: Xaxis J3, Battery:smd_pad_10, F.Cu at (506.6, 81.4)
- added J9: Xaxis J4, Battery:smd_pad_10, F.Cu at (506.6, 85.5)
- added LS1: CMT-8530S-SMT, Capacitor_SMD:CUI_CMT-8530S-SMT, F.Cu at (446.5, 75.2)
- added LS2: CMT-8530S-SMT, Capacitor_SMD:CUI_CMT-8530S-SMT, F.Cu at (446.5, 86.3)
- added LS3: CMT-8530S-SMT, Capacitor_SMD:CUI_CMT-8530S-SMT, F.Cu at (446.5, 97.3)
- added LS4: CMT-8530S-SMT, Capacitor_SMD:CUI_CMT-8530S-SMT, F.Cu at (446.5, 108.4)
- added Q4: BC847, Package_TO_SOT_SMD:SOT-23, F.Cu at (533.6, 97.5)
- added Q5: BC847, Package_TO_SOT_SMD:SOT-23, F.Cu at (533.6, 101.9)
- added Q8: BC847, Package_TO_SOT_SMD:SOT-23, F.Cu at (533.6, 106.4)
- added Q9: BC847, Package_TO_SOT_SMD:SOT-23, F.Cu at (533.6, 110.8)
- added R50: 1K, Resistor_SMD:R_0402_1005Metric, F.Cu at (440.5, 48.6)
- added R51: 1K, Resistor_SMD:R_0402_1005Metric, F.Cu at (440.5, 50.6)
- added R52: 0, Resistor_SMD:R_0402_1005Metric, F.Cu at (520.7, 80.3)
- added R58: 0, Resistor_SMD:R_0402_1005Metric, F.Cu at (520.7, 92.3)
- added R59: 0, Resistor_SMD:R_0402_1005Metric, F.Cu at (520.7, 94.3)
- added R60: 0, Resistor_SMD:R_0402_1005Metric, F.Cu at (523.6, 80.3)
- added R61: 0, Resistor_SMD:R_0402_1005Metric, F.Cu at (523.6, 82.3)
- added R62: 0, Resistor_SMD:R_0402_1005Metric, F.Cu at (523.6, 84.3)
- added R63: 0, Resistor_SMD:R_0402_1005Metric, F.Cu at (523.6, 86.3)
- added R64: 0, Resistor_SMD:R_0402_1005Metric, F.Cu at (523.6, 88.3)
- added R65: 0, Resistor_SMD:R_0402_1005Metric, F.Cu at (523.6, 90.3)
- added R66: 0, Resistor_SMD:R_0402_1005Metric, F.Cu at (523.6, 92.3)
- added R67: 0, Resistor_SMD:R_0402_1005Metric, F.Cu at (523.6, 94.3)
- added R68: 0, Resistor_SMD:R_0402_1005Metric, F.Cu at (526.5, 80.3)
- added R69: 0, Resistor_SMD:R_0402_1005Metric, F.Cu at (526.5, 82.3)
- added R70: 0, Resistor_SMD:R_0402_1005Metric, F.Cu at (526.5, 84.3)
- added R71: 0, Resistor_SMD:R_0402_1005Metric, F.Cu at (526.5, 86.3)
- added R72: 0, Resistor_SMD:R_0402_1005Metric, F.Cu at (526.5, 88.3)
- added R73: 0, Resistor_SMD:R_0402_1005Metric, F.Cu at (526.5, 90.3)
- added R74: 0, Resistor_SMD:R_0402_1005Metric, F.Cu at (526.5, 92.3)
- added R75: 0, Resistor_SMD:R_0402_1005Metric, F.Cu at (526.5, 94.3)
- added R76: 0, Resistor_SMD:R_0402_1005Metric, F.Cu at (529.4, 80.3)
- added R77: 0, Resistor_SMD:R_0402_1005Metric, F.Cu at (529.4, 82.3)
- added R78: 0, Resistor_SMD:R_0402_1005Metric, F.Cu at (529.4, 84.3)
- added R90: 0, Resistor_SMD:R_0402_1005Metric, F.Cu at (529.4, 86.3)
- added R91: 1K, Resistor_SMD:R_0402_1005Metric, F.Cu at (529.4, 88.3)
- added R92: 0, Resistor_SMD:R_0402_1005Metric, F.Cu at (529.4, 90.3)
- added R93: 220, Resistor_SMD:R_0402_1005Metric, F.Cu at (529.4, 92.3)
- added R94: 220, Resistor_SMD:R_0402_1005Metric, F.Cu at (529.4, 94.3)
- added R95: 0, Resistor_SMD:R_0402_1005Metric, F.Cu at (481.1, 112.1)
- added R96: 1K, Resistor_SMD:R_0402_1005Metric, F.Cu at (481.1, 114.0)
- added SW7: SW_SPDT, Button_Switch_THT:SW_Slide_1P2T_CK_OS102011MS2Q, F.Cu at (523.2, 98.8)
- added SW8: SW_SPDT, Button_Switch_THT:SW_Slide_1P2T_CK_OS102011MS2Q, F.Cu at (523.2, 105.2)
- added U11: Ai-Thinker-Ra-02, RF_Module:Ai-Thinker-Ra-01-LoRa, F.Cu at (471.8, 79.2)
- added U12: Ai-Thinker-Ra-02, RF_Module:Ai-Thinker-Ra-01-LoRa, F.Cu at (471.8, 98.3)
- added U13: MPU-6050, Button_Switch_SMD:QFN50P400X400X95-24N, F.Cu at (513.6, 100.3)
- added U14: ~, Audio_Module:5v_usbbuck, F.Cu at (408.4, 41.6)
- added U15: ~, Audio_Module:buck 5v, F.Cu at (408.4, 84.2)
- added U17: ~, Audio_Module:5v_usbbuck, F.Cu at (395.3, 176.4)
- added U2: RASPBERRY_PI_4B_4GB, Button_Switch_SMD:MODULE_RASPBERRY_PI_4B_4GB, F.Cu at (490.1, 38.9)
- added U21: ~, Audio_Module:5v_usbbuck, F.Cu at (419.7, 176.4)
- added U22: ESP32-WROOM-32D, RF_Module:ESP32-WROOM-32D, F.Cu at (356.9, 167.3)
- added U23: ESP32-WROOM-32D, RF_Module:ESP32-WROOM-32D, F.Cu at (356.9, 209.8)
- added U24: ESP32-WROOM-32D, RF_Module:ESP32-WROOM-32D, F.Cu at (356.9, 252.4)
- C24, C25, C26, C27, C28, C29, C33, C34, C35: value 0.1uF -> 100uF; footprint Capacitor_SMD:C_0402_1005Metric -> Battery:CAPAE830X1000N
- R22, R23, R27, R38, R53, R54, R55, R57: value 1K -> 0
- R25, R30, R48: value 0 -> 1K
- U1, U3, U4, U5, U7: value AP2112K-3.3 -> AMS1117-3.3; footprint Package_TO_SOT_SMD:SOT-23-5 -> Package_TO_SOT_SMD:SOT-223-3_TabPin2
- U10, U6, U8: value ESP32-WROOM-32D -> ~; footprint RF_Module:ESP32-WROOM-32D -> Audio_Module:buck 5v
- U16: value AP2112K-3.3 -> ~; footprint Package_TO_SOT_SMD:SOT-23-5 -> Audio_Module:buck 5v
- U9: value ESP32-WROOM-32D -> AMS1117-3.3; footprint RF_Module:ESP32-WROOM-32D -> Package_TO_SOT_SMD:SOT-223-3_TabPin2
- moved J6 503.1 mm to (558.0, 35.4)
- moved U7 497.3 mm to (547.3, 47.3)
- moved J1 488.9 mm to (558.0, 15.4)
- moved R15 483.9 mm to (571.1, 11.1)
- moved R16 483.9 mm to (571.1, 13.1)
- moved R17 483.9 mm to (571.1, 15.1)
- moved R18 483.9 mm to (571.1, 17.1)
- moved R19 483.9 mm to (571.1, 19.1)
- moved R20 483.9 mm to (571.1, 21.1)
- moved R21 483.9 mm to (571.1, 23.1)
- moved R1 483.9 mm to (565.3, 11.1)
- moved R2 483.9 mm to (565.3, 13.1)
- moved R3 483.9 mm to (565.3, 15.1)
- moved R4 483.9 mm to (565.3, 17.1)
- moved R5 483.9 mm to (565.3, 19.1)
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Connections:
- net /UART Bridge/RX1 renamed /RX1
- net /UART Bridge/RX3 renamed /RX3
- net /UART Bridge/TX1 renamed /TX1
- net /UART Bridge/TX3 renamed /TX3
- C24 pad 1: GND -> Vin
- C24 pad 2: /SoC/EN1 -> GND
- C25 pad 1: GND -> +5V
- C25 pad 2: Net-(U6-VDD) -> GND
- C26 pad 1: GND -> 4S
- C26 pad 2: /SoC/IO01 -> GND
- C27 pad 1: GND -> Vin
- C27 pad 2: /SoC/EN2 -> GND
- C28 pad 1: GND -> +5V
- C28 pad 2: Net-(U8-VDD) -> GND
- C29 pad 1: GND -> 4S
- C29 pad 2: /SoC/IO02 -> GND
- C30 pad 2: /EN -> Net-(U11-VDD)
- C31 pad 2: Net-(U9-VDD) -> Net-(U12-VDD)
- C32 pad 1: GND -> +3.3V
- C32 pad 2: /IO0 -> GND
- C33 pad 1: GND -> Vin
- C33 pad 2: /SoC/EN3 -> GND
- C34 pad 1: GND -> +5V
- C34 pad 2: Net-(U10-VDD) -> GND
- C35 pad 1: GND -> 4S
- C35 pad 2: /SoC/IO03 -> GND
- D17 pad 1: /UART Bridge/RX2 -> /RX2
- D18 pad 1: /UART Bridge/TX2 -> /TX2
- J1 pad A6: /Power Supply/D1+ -> /D1+
- J1 pad A7: /Power Supply/D1- -> /D1-
- J1 pad B6: /Power Supply/D1+ -> /D1+
- J1 pad B7: /Power Supply/D1- -> /D1-
- J5 pad A6: /Power Supply/D2+ -> /D2+
- J5 pad A7: /Power Supply/D2- -> /D2-
- J5 pad B6: /Power Supply/D2+ -> /D2+
- J5 pad B7: /Power Supply/D2- -> /D2-
- J6 pad A6: /Power Supply/D3+ -> /D3+
- J6 pad A7: /Power Supply/D3- -> /D3-
- J6 pad B6: /Power Supply/D3+ -> /D3+
- J6 pad B7: /Power Supply/D3- -> /D3-
- Q11 pad 3: /UART Bridge/EN2 -> /EN2
- Q12 pad 3: /UART Bridge/IO02 -> /IO02
- Q13 pad 3: /UART Bridge/EN3 -> /EN3
- Q14 pad 3: /UART Bridge/IO03 -> /IO03
- Q6 pad 3: /UART Bridge/EN1 -> /EN1
- Q7 pad 3: /UART Bridge/IO01 -> /IO01
- R13 pad 2: Net-(U4-VOUT) -> Net-(U3-VO)
- R20 pad 2: Net-(U16-VOUT) -> Net-(U5-VO)
- R22 pad 1: /SoC/SDA1 -> +5V
- R22 pad 2: +3.3V -> Net-(U6-5V)
- R23 pad 1: +3.3V -> +5V
- R23 pad 2: /SoC/SCL1 -> Net-(U15-5V)
- R24 pad 1: /SoC/EN1 -> /SDA1
- R25 pad 1: Net-(U6-VDD) -> +3.3V
- R25 pad 2: +3.3V -> /SCL1
- R26 pad 1: /SoC/IO01 -> /EN1
- R27 pad 1: /SoC/SDA2 -> Net-(U22-VDD)
- R28 pad 1: +3.3V -> /IO01
- R28 pad 2: /SoC/SCL2 -> +3.3V
- R29 pad 1: /SoC/EN2 -> /SDA1
- R30 pad 1: Net-(U8-VDD) -> /SDAx
- R31 pad 1: /SoC/IO02 -> +3.3V
- R31 pad 2: +3.3V -> /SCL1
- R33 pad 1: /SoC/SDA3 -> +3.3V
- R33 pad 2: +3.3V -> /SCLx
- R34 pad 1: +3.3V -> /EN2
- R34 pad 2: /SoC/SCL3 -> +3.3V
- R38 pad 1: /SoC/EN3 -> Net-(U23-VDD)
- R45 pad 1: /UART Bridge/TX2 -> /TX2
- R46 pad 2: /UART Bridge/RX2 -> /RX2
- R48 pad 1: Net-(U10-VDD) -> /IO02
- R49 pad 1: /SoC/IO03 -> /SDA1
- R53 pad 1: /SDA -> Net-(U12-VDD)
- R54 pad 1: +3.3V -> Net-(J2-Pin_6)
- R54 pad 2: /SCL -> /Aa
- R55 pad 1: /EN -> Net-(J3-Pin_6)
- R55 pad 2: +3.3V -> /Ab
- R56 pad 1: Net-(U9-VDD) -> Net-(J3-Pin_5)
- R57 pad 1: /IO0 -> +3.3V
- R57 pad 2: +3.3V -> Net-(J4-Pin_1)
- R6 pad 2: Net-(U1-VOUT) -> Net-(U1-VO)
- SW1 pad 2: /SoC/EN1 -> /EN1
- SW2 pad 2: /SoC/IO01 -> /IO01
- SW3 pad 2: /SoC/EN2 -> /EN2
- SW4 pad 2: /SoC/IO02 -> /IO02
- SW5 pad 2: /SoC/EN3 -> /EN3
- SW6 pad 2: /SoC/IO03 -> /IO03
- U1 pad 1: VBUS -> GND
- U1 pad 2: GND -> Net-(U1-VO)
- U10 pad 1: GND -> 4S
- U10 pad 2: Net-(U10-VDD) -> GND
- U10 pad 3: /SoC/EN3 -> GND
- U10 pad 4: unconnected-(U10-SENSOR_VP-Pad4) -> +5V
- U16 pad 1: VBUS -> 4S
- U16 pad 3: VBUS -> GND
- U16 pad 4: unconnected-(U16-NC-Pad4) -> Net-(U15-5V)
- U18 pad 4: /UART Bridge/D1+ -> /D1+
- U18 pad 5: /UART Bridge/D1- -> /D1-
- U19 pad 4: /UART Bridge/D2+ -> /D2+
- U19 pad 5: /UART Bridge/D2- -> /D2-
- U20 pad 4: /UART Bridge/D3+ -> /D3+
- U20 pad 5: /UART Bridge/D3- -> /D3-
- U3 pad 1: VBUS -> GND
- U3 pad 2: GND -> Net-(U3-VO)
- U4 pad 1: VBUS -> GND
- U4 pad 2: GND -> Net-(U3-VO)
- U5 pad 1: VBUS -> GND
- U5 pad 2: GND -> Net-(U5-VO)
- U6 pad 1: GND -> 4S
- U6 pad 2: Net-(U6-VDD) -> GND
- U6 pad 3: /SoC/EN1 -> GND
- U6 pad 4: unconnected-(U6-SENSOR_VP-Pad4) -> Net-(U6-5V)
- U7 pad 1: VBUS -> GND
- U7 pad 2: GND -> Net-(U5-VO)
- U8 pad 1: GND -> 4S
- U8 pad 2: Net-(U8-VDD) -> GND
- U8 pad 3: /SoC/EN2 -> GND
- U8 pad 4: unconnected-(U8-SENSOR_VP-Pad4) -> Net-(U6-5V)
- U9 pad 2: Net-(U9-VDD) -> Net-(U1-VO)
- U9 pad 3: /EN -> VBUS

Commit message: update remote_v2
Parts:
- moved U2 290.4 mm to (199.6, 40.9)
Changed lines of the file:
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@@
   )
   (footprint "Button_Switch_SMD:MODULE_RASPBERRY_PI_4B_4GB" (layer "F.Cu")
-    (at 490.062 38.91)
+    (at 199.6195 40.915)
     (property "Availability" "In Stock")
     (property "Check_prices" "https://www.snapeda.com/parts/RASPBERRY%20PI%204B/4GB/Raspberry+Pi/view-part/?ref=eda")

Commit message: update watch_v3
Parts:
- C47, C48: footprint Capacitor_SMD:C_0402_1005Metric -> Battery:CAPAE830X1000N
- J27: footprint Connector_PinHeader_2.54mm:PinHeader_1x10_P2.54mm_Vertical -> Button_Switch_SMD:solder_10
- U2: value RASPBERRY_PI_4B_4GB -> RASPBERRY_PI_5
- moved J25 469.0 mm to (63.8, 131.8)
- moved R94 413.9 mm to (119.1, 39.6)
- moved J6 377.2 mm to (185.7, 95.5), turned to 90 degrees
- moved U23 305.0 mm to (566.5, -11.8)
- moved J26 300.5 mm to (69.6, -18.7)
- moved U11 260.9 mm to (212.6, 109.2), turned to 180 degrees
- moved U22 250.9 mm to (136.8, 46.9)
- moved U24 248.5 mm to (141.9, 127.9), turned to 180 degrees
- moved U12 226.8 mm to (318.6, -69.0), turned to 180 degrees
- moved U6 205.4 mm to (661.0, 127.0)
- moved J27 184.6 mm to (220.1, -61.8)
- moved U2 126.8 mm to (76.2, 70.1)
- moved U14 79.3 mm to (468.6, -10.0)
Other:
- board outline added: 99.7 x 100 mm

Commit message: updating watch_v3
Parts:
- removed C62, C70, C72, C82, C83, C85, C86, C88: 100uF, Battery:CAPAE830X1000N
- removed D11, D12, D8: 1N4148, Diode_SMD:D_SOD-323
- removed LS2, LS3, LS4: CMT-8530S-SMT, Capacitor_SMD:CUI_CMT-8530S-SMT
- removed Q5, Q8, Q9: BC847, Package_TO_SOT_SMD:SOT-23
- added J28: Mode1, Battery:smd_pad_10, F.Cu at (92.9, 128.8)
- added J29: Mode3, Battery:smd_pad_10, F.Cu at (92.9, 133.0)
- added J30: Mode2, Battery:smd_pad_10, F.Cu at (92.9, 137.2)
- added J31: Mode4, Battery:smd_pad_10, F.Cu at (92.9, 141.3)
- added R100: 0, Resistor_SMD:R_0402_1005Metric, F.Cu at (89.7, 149.0)
- added R101: 0, Resistor_SMD:R_0402_1005Metric, F.Cu at (89.7, 151.0)
- added R97: 0, Resistor_SMD:R_0402_1005Metric, F.Cu at (89.7, 143.0)
- added R98: 0, Resistor_SMD:R_0402_1005Metric, F.Cu at (89.7, 145.0)
- added R99: 0, Resistor_SMD:R_0402_1005Metric, F.Cu at (89.7, 147.0)
- J17, J25: footprint Button_Switch_SMD:AMASS_XT60-M -> Battery:AMASS_XT60PW-M
- moved U6 632.6 mm to (33.7, 208.2)
- moved D1 610.6 mm to (-15.9, 211.7)
- moved D3 610.6 mm to (-15.9, 216.3)
- moved D5 610.6 mm to (-15.9, 220.8)
- moved J1 610.6 mm to (-23.7, 200.8)
- moved J5 610.6 mm to (-23.7, 210.8)
- moved R1 610.6 mm to (-16.4, 196.5)
- moved R15 610.6 mm to (-10.6, 196.5)
- moved R16 610.6 mm to (-10.6, 198.5)
- moved R17 610.6 mm to (-10.6, 200.5)
- moved R18 610.6 mm to (-10.6, 202.5)
- moved R19 610.6 mm to (-10.6, 204.5)
- moved R2 610.6 mm to (-16.4, 198.5)
- moved R20 610.6 mm to (-10.6, 206.5)
- moved R21 610.6 mm to (-10.6, 208.5)
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Connections:
- R75 pad 1: +3.3V -> /Mode1
- U23 pad 13: /BuzzJ4 -> /Mode3
- U23 pad 14: /BuzzJ2 -> /Mode1
- U23 pad 16: /BuzzJ3 -> /Mode2
- U23 pad 23: unconnected-(U23-IO15-Pad23) -> /Mode4
Other:
- board outline removed
