File: PCB/Remote_V2/remote_v2.kicad_pcb (KiCad board)
At the start: 2 copper layers, 151.3 x 122.6 mm, 130 parts, among them J10 Yaxis J1, J11 Yaxis J2, J12 Yaxis J3, J13 Yaxis J4, J17 XT60-M, J2 ADS1115 A1, J24 5V, J25 XT60-M, J26 UART RASP, J28 Mode1, J29 Mode3, J3 ADS1115 A2, J30 Mode2, J31 Mode4, J32 Conn_01x07_Pin, J33 Conn_01x07_Pin, J4 Xaxis J1, J6 Conn_01x07_Pin, J7 Xaxis J2, J8 Xaxis J3, J9 Xaxis J4, Q1 AO3401A, Q4 BC847, SW1 SW_DPST_x2, SW2 SW_DPST_x2, SW3 SW_DPST_x2, SW4 SW_DPST_x2, SW5 SW_DPST_x2, SW6 SW_DPST_x2, SW7 SW_SPDT, SW8 SW_SPDT, U1 AMS1117-3.3, U11 Ai-Thinker-Ra-02, U12 Ai-Thinker-Ra-02, U13 MPU-6050, U2 RASPBERRY_PI_5, U22 ESP32-WROOM-32D, U23 ESP32-WROOM-32D, U24 ESP32-WROOM-32D, U3 AMS1117-3.3, U4 AMS1117-3.3, U9 AMS1117-3.3

Commit message: updating PCB design
Parts:
- added R3: 0, Resistor_SMD:R_0402_1005Metric, F.Cu at (126.0, 125.8)
- added REF**: MountingHole_3.2mm_M3_DIN965, MountingHole:MountingHole_3.2mm_M3_DIN965, F.Cu at (127.0, 59.1)
- added REF**: MountingHole_3.2mm_M3_DIN965, MountingHole:MountingHole_3.2mm_M3_DIN965, F.Cu at (204.1, 136.3)
- added REF**: MountingHole_3.2mm_M3_DIN965, MountingHole:MountingHole_3.2mm_M3_DIN965, F.Cu at (174.4, 56.0)
- added REF**: MountingHole_3.2mm_M3_DIN965, MountingHole:MountingHole_3.2mm_M3_DIN965, F.Cu at (61.1, 157.9)
Connections:
- C3 pad 2: Net-(Q1-D) -> VBUS
Routing:
- net VBUS: track 35.3 -> 44.7 mm, vias 0 -> 1
- net /Vx4: track 51.7 -> 49.8 mm
- net Net-(Q1-D): track 11.0 -> 9.28 mm
- net +5V: track 194.9 -> 195.9 mm
- net GND: track 1186.1 -> 1185.4 mm
- net /Vy4: track 35.9 -> 35.3 mm

Commit message: updating PCB
Parts:
- moved D1 1.04 mm to (131.8, 124.6)
Routing:
- net Net-(Q1-D): track 9.28 -> 10.4 mm
- net Net-(Q1-G): track 41.5 -> 42.3 mm
Changed lines of the file:
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@@
   )
   (footprint "Button_Switch_SMD:P25_DO-214AC_SMA" (layer "B.Cu")
-    (at 132.8225 124.49 180)
+    (at 131.79 124.59 180)
     (descr "Diode SMA (DO-214AC)")
     (tags "SMA (DO-214AC)")
@@
   (segment (start 148.1 125.29) (end 146.4 123.59) (width 0.16) (layer "B.Cu") (net 3))
   (segment (start 132.27 119.45) (end 132.27 121.67) (width 0.25) (layer "B.Cu") (net 3))
+  (segment (start 132.75 122.15) (end 132.93 122.33) (width 0.25) (layer "B.Cu") (net 3))
   (segment (start 132.27 116.33) (end 131.91 115.97) (width 0.25) (layer "B.Cu") (net 3))
   (segment (start 132.27 121.67) (end 132.75 122.15) (width 0.25) (layer "B.Cu") (net 3))
+  (segment (start 131.79 123.11) (end 132.75 122.15) (width 0.25) (layer "B.Cu") (net 3))
+  (segment (start 131.79 124.59) (end 131.79 123.11) (width 0.25) (layer "B.Cu") (net 3))
   (segment (start 142.56 116.48) (end 140.13 116.48) (width 0.16) (layer "B.Cu") (net 3))
   (segment (start 148.1 125.52) (end 148.1 125.29) (width 0.16) (layer "B.Cu") (net 3))
@@
   (segment (start 131.91 115.97) (end 131.91 114.9) (width 0.16) (layer "B.Cu") (net 3))
   (segment (start 127.56 120.125) (end 127.56 121.74) (width 0.25) (layer "B.Cu") (net 3))
-  (segment (start 132.75 124.4175) (end 132.8225 124.49) (width 0.25) (layer "B.Cu") (net 3))
   (segment (start 128.245 119.44) (end 127.56 120.125) (width 0.25) (layer "B.Cu") (net 3))
   (segment (start 131.91 114.9) (end 132.27 114.54) (width 0.16) (layer "B.Cu") (net 3))
-  (segment (start 132.75 122.15) (end 132.75 124.4175) (width 0.25) (layer "B.Cu") (net 3))
   (segment (start 132.27 119.45) (end 132.27 116.33) (width 0.25) (layer "B.Cu") (net 3))
-  (segment (start 128.8225 124.49) (end 128.8225 127.12) (width 0.25) (layer "B.Cu") (net 4))
-  (segment (start 130.12 118.49) (end 130.12 123.1925) (width 0.25) (layer "B.Cu") (net 4))
-  (segment (start 128.8225 127.12) (end 128.7425 127.2) (width 0.25) (layer "B.Cu") (net 4))
-  (segment (start 130.12 123.1925) (end 128.8225 124.49) (width 0.25) (layer "B.Cu") (net 4))
+  (segment (start 128.7425 125.5425) (end 127.79 124.59) (width 0.25) (layer "B.Cu") (net 4))
+  (segment (start 130.12 118.49) (end 130.12 122.73) (width 0.25) (layer "B.Cu") (net 4))
+  (segment (start 128.26 124.59) (end 127.79 124.59) (width 0.25) (layer "B.Cu") (net 4))
+  (segment (start 130.12 122.73) (end 128.26 124.59) (width 0.25) (layer "B.Cu") (net 4))
+  (segment (start 128.69 127.1475) (end 128.7425 127.2) (width 0.25) (layer "B.Cu") (net 4))
+  (segment (start 128.7425 127.2) (end 128.7425 125.5425) (width 0.25) (layer "B.Cu") (net 4))
   (segment (start 133.84 138.41) (end 144.98 138.41) (width 0.16) (layer "F.Cu") (net 5))
   (segment (start 154.615 64.345) (end 154.615 60.925) (width 0.16) (layer "F.Cu") (net 5))
