File: PCB/Remote_V2/remote_v2.kicad_sch (KiCad schematic)
At the start: 90 parts, among them J10 Yaxis J1, J11 Yaxis J2, J12 Yaxis J3, J13 Yaxis J4, J14 ICSP1, J15 ICSP2, J16 ICSP3, J17 5V, J18 Peri Soc 1, J19 Peri Soc 2, J2 ADS1115 A1, J20 Peri Soc 3, J21 UART Soc 1, J22 UART Soc 2, J23 UART Soc 3, J3 ADS1115 A2, J4 Xaxis J1, J7 Xaxis J2, J8 Xaxis J3, J9 Xaxis J4, Q4 BC847, Q5 BC847, Q8 BC847, Q9 BC847, SW7 SW_SPDT, U11 Ai-Thinker-Ra-02, U12 Ai-Thinker-Ra-02, U13 MPU-6050, U2 RASPBERRY_PI_4B_4GB

Commit message: remote_v2 update
Parts:
- removed C54, C55: 100uF, Capacitor_SMD:C_0402_1005Metric, symbol Device:C
- removed J17: 5V, symbol Connector:Conn_01x02_Pin
- added C54, C55, C56, C57: 100uF, Battery:CAPAE830X1000N, symbol UWT1V101MCL1GS:UWT1V101MCL1GS
- added D13, D14: LED, LED_SMD:LED_0402_1005Metric, symbol Device:LED
- added J24: 5V, Button_Switch_SMD:solder_motor, symbol Connector:Conn_01x02_Pin
- added J25: XT60-M, Button_Switch_SMD:AMASS_XT60-M, symbol XT60-M:XT60-M
- added J26: UART RASP, Button_Switch_SMD:solder_pad_4, symbol Connector:Conn_01x04_Pin
- added J27: RASP Peripheral, Connector_PinHeader_2.54mm:PinHeader_1x10_P2.54mm_Vertical, symbol Connector:Conn_01x10_Pin
- added R93, R94: 220, Resistor_SMD:R_0402_1005Metric, symbol Device:R
- added SW8: SW_SPDT, Button_Switch_THT:SW_Slide_1P2T_CK_OS102011MS2Q, symbol Switch:SW_SPDT
- J10, J11, J12, J13, J4, J7, J8, J9: footprint (none) -> Battery:smd_pad_10
- J14, J15, J16, J18, J19, J20, J21, J22, J23: footprint (none) -> Button_Switch_SMD:solder_pad_4
- J2, J3: footprint (none) -> Connector_PinHeader_2.54mm:PinHeader_1x10_P2.54mm_Vertical
Connections:
- net +3.3V: now also J26.1 (Pin_1), J27.1 (Pin_1)
- net +5V: now also C56.1, C57.1
- net 5V: now also J24.2 (Pin_2), J25.P (POS)
- net GND: now also C54.2, C55.2, C56.2, C57.2, D13.1 (K), D14.1 (K), J24.1 (Pin_1), J25.N (NEG), J26.4 (Pin_4), J27.10 (Pin_10)
- net SCL1: now also R93.1
- net SDA1: now also R94.2
- net ce0: now also J27.5 (Pin_5)
- net ce1: now also J27.6 (Pin_6)
- net gp17: now also J27.2 (Pin_2)
- net gp18: now also J27.4 (Pin_4)
- net gp27: now also J27.3 (Pin_3)
- net miso: now also J27.9 (Pin_9)
- net mosi: now also J27.8 (Pin_8)
- net rx: now also J26.3 (Pin_3)
- net sclk: now also J27.7 (Pin_7)
- net tx: now also J26.2 (Pin_2)
- net gp22: no longer names the net of U2.15 (GPIO22/GPIO_GEN3)
- new net: D14.2 (A), R94.1
- new net: D13.2 (A), R93.2
- new net 4S: C54.1, C55.1, SW8.1 (A)
- new net Vin: SW8.2 (B)
- no-connect marks 38 -> 39
Other:
- removed sheet SoC
- added sheet 5v~buck1 (buck.kicad_sch)
- added sheet SoC1 (soc.kicad_sch)
- sheet Power Supply ports: added 3.3V, 5V, D1+, D1-, D2+, D2-, D3+, D3-, GND, VBUS, VCCQ; removed none
- sheet UART Bridge ports: added D1+, D1-, D2+, D2-, D3+, D3-, EN1, EN2, EN3, GND, IO01, IO02, IO03, RX1, RX2, RX3, TX1, TX2, TX3, VBUS; removed none
- note added: "4S Switch"
- note added: "5V POWER IN"
- note added: "5V Switch"
- note added: "5v Buck"
- note added: "ADC I2C"
- note added: "Buzzer Indicator"
- note added: "ICSP"
- note added: "Joystick Connector"
- note added: "LORA SX1278 RA-02"
- note added: "MPU-6050"
- note added: "Peri. RASPI"
- note added: "Peripheral Port"
- note added: "Power&UART Unit"
- note added: "Rasp 5 Board"
- note added: "SOC"
- note added: "UART1 PORT"
- note added: "UTILITY REMOTE"
- moved on the sheet: SW7

Commit message: update remote_v2
Parts:
- U2: value RASPBERRY_PI_4B_4GB -> RASPBERRY_PI_5
Other:
- note added: "REMOTE"
- note added: "UTILITY"
- note removed: "UTILITY REMOTE"
- moved on the sheet: J27
Changed lines of the file:
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@@
     (stroke (width 0) (type default))
   )
-  (wire (pts (xy 257.175 63.5) (xy 257.175 66.04))
+  (wire (pts (xy 257.175 63.5) (xy 257.175 70.485))
     (stroke (width 0) (type default))
   )
@@
     (stroke (width 0) (type default))
   )
-  (wire (pts (xy 262.89 63.5) (xy 262.89 65.405))
+  (wire (pts (xy 262.89 63.5) (xy 262.89 72.39))
     (stroke (width 0) (type default))
   )
@@
     (stroke (width 0) (type default))
   )
-  (wire (pts (xy 259.08 63.5) (xy 259.08 66.675))
+  (wire (pts (xy 259.08 63.5) (xy 259.08 68.58))
     (stroke (width 0) (type default))
   )
@@
     (stroke (width 0) (type default))
   )
-  (wire (pts (xy 264.795 63.5) (xy 264.795 66.04))
+  (wire (pts (xy 264.795 63.5) (xy 264.795 70.485))
     (stroke (width 0) (type default))
   )
@@
     (stroke (width 0) (type default))
   )
-  (wire (pts (xy 260.985 63.5) (xy 260.985 66.04))
+  (wire (pts (xy 260.985 63.5) (xy 260.985 67.31))
     (stroke (width 0) (type default))
   )
@@
     (stroke (width 0) (type default))
   )
-  (rectangle (start 208.28 104.14) (end 282.575 165.735)
+  (rectangle (start 208.28 104.14) (end 282.575 161.29)
     (stroke (width 0.3) (type dash) (color 255 44 9 1))
     (fill (type none))
@@
     (fill (type none))
   )
-  (rectangle (start 169.545 104.14) (end 202.565 165.735)
+  (rectangle (start 169.545 104.14) (end 202.565 165.1)
     (stroke (width 0.3) (type dash) (color 255 44 9 1))
     (fill (type none))
@@
     (fill (type none))
   )
-  (rectangle (start 238.125 12.7) (end 283.21 67.31)
+  (rectangle (start 238.125 12.7) (end 283.21 73.66)
     (stroke (width 0.3) (type dash) (color 255 44 9 1))
     (fill (type none))
@@
     (fill (type none))
   )
-  (rectangle (start 204.47 22.225) (end 229.87 52.705)
+  (rectangle (start 204.47 15.875) (end 229.87 46.355)
     (stroke (width 0.3) (type dash) (color 255 44 9 1))
     (fill (type none))
@@
     (fill (type none))
   )
-  (text "UTILITY REMOTE\n" (at 281.305 77.47 0)
+  (text "UTILITY\n\n" (at 235.585 65.405 0)
     (effects (font (size 6 6) (thickness 1.6) bold (color 253 61 255 1)) (justify right bottom))
   )
@@
     (effects (font (size 1.27 1.27) bold (color 0 28 255 1)) (justify left bottom))
   )
-  (text "Peri. RASPI\n" (at 205.74 25.4 0)
+  (text "Peri. RASPI\n" (at 205.74 19.05 0)
     (effects (font (size 1.27 1.27) bold (color 0 28 255 1)) (justify left bottom))
   )
@@
     (effects (font (size 1.27 1.27) bold (color 0 28 255 1)) (justify left bottom))
   )
+  (text "\nREMOTE\n" (at 236.855 64.77 0)
+    (effects (font (size 6 6) (thickness 1.6) bold (color 253 61 255 1)) (justify right bottom))
+  )
   (text "ICSP\n" (at 56.515 142.875 0)
     (effects (font (size 1.27 1.27) bold (color 0 28 255 1)) (justify left bottom))
@@
     (effects (font (size 1.27 1.27)) (justify left bottom))
   )
-  (label "ce0" (at 221.615 36.83 180) (fields_autoplaced)
+  (label "ce0" (at 221.615 30.48 180) (fields_autoplaced)
     (effects (font (size 1 1)) (justify right bottom))
   )
@@
     (effects (font (size 1 1)) (justify right bottom))
   )
-  (label "ce1" (at 221.615 39.37 180) (fields_autoplaced)
+  (label "ce1" (at 221.615 33.02 180) (fields_autoplaced)
     (effects (font (size 1 1)) (justify right bottom))
   )
@@
     (effects (font (size 1 1)) (justify right bottom))
   )
-  (label "BuzzJ4" (at 259.08 66.675 0) (fields_autoplaced)
+  (label "BuzzJ4" (at 259.08 68.58 0) (fields_autoplaced)
     (effects (font (size 1 1)) (justify left bottom))
   )
@@
     (effects (font (size 1 1)) (justify left bottom))
   )
-  (label "sclk" (at 221.615 41.91 180) (fields_autoplaced)
+  (label "sclk" (at 221.615 35.56 180) (fields_autoplaced)
     (effects (font (size 1 1)) (justify right bottom))
   )
@@
     (effects (font (size 1 1)) (justify right bottom))
   )
-  (label "S1-14" (at 264.795 66.04 0) (fields_autoplaced)
+  (label "S1-14" (at 264.795 70.485 0) (fields_autoplaced)
     (effects (font (size 1 1)) (justify left bottom))
   )
@@
     (effects (font (size 1 1)) (justify left bottom))
   )
-  (label "miso" (at 221.615 46.99 180) (fields_autoplaced)
+  (label "miso" (at 221.615 40.64 180) (fields_autoplaced)
     (effects (font (size 1 1)) (justify right bottom))
   )
@@
     (effects (font (size 1 1)) (justify right bottom))
   )
-  (label "S1-13" (at 262.89 65.405 0) (fields_autoplaced)
+  (label "S1-13" (at 262.89 72.39 0) (fields_autoplaced)
     (effects (font (size 1 1)) (justify left bottom))
   )
@@
     (effects (font (size 1 1)) (justify left bottom))
   )
-  (label "TX2" (at 257.175 66.04 0) (fields_autoplaced)
+  (label "TX2" (at 257.175 70.485 0) (fields_autoplaced)
     (effects (font (size 1 1)) (justify left bottom))
   )
@@
     (effects (font (size 1 1)) (justify right bottom))
   )
-  (label "gp17" (at 221.615 29.21 180) (fields_autoplaced)
+  (label "gp17" (at 221.615 22.86 180) (fields_autoplaced)
     (effects (font (size 1 1)) (justify right bottom))
   )
@@
     (effects (font (size 1.27 1.27)) (justify left bottom))
   )
-  (label "TX3" (at 260.985 66.04 0) (fields_autoplaced)
+  (label "TX3" (at 260.985 67.31 0) (fields_autoplaced)
     (effects (font (size 1 1)) (justify left bottom))
   )
@@
     (effects (font (size 1.27 1.27)) (justify left bottom))
   )
-  (label "gp18" (at 221.615 34.29 180) (fields_autoplaced)
+  (label "gp18" (at 221.615 27.94 180) (fields_autoplaced)
     (effects (font (size 1 1)) (justify right bottom))
   )
@@
     (effects (font (size 1 1)) (justify right bottom))
   )
-  (label "gp27" (at 221.615 31.75 180) (fields_autoplaced)
+  (label "gp27" (at 221.615 25.4 180) (fields_autoplaced)
     (effects (font (size 1 1)) (justify right bottom))
   )
@@
     (effects (font (size 1 1)) (justify right bottom))
   )
-  (label "mosi" (at 221.615 44.45 180) (fields_autoplaced)
+  (label "mosi" (at 221.615 38.1 180) (fields_autoplaced)
     (effects (font (size 1 1)) (justify right bottom))
   )
@@
     )
   )
-  (symbol (lib_id "power:GND") (at 221.615 49.53 270) (unit 1)
+  (symbol (lib_id "power:GND") (at 221.615 43.18 270) (unit 1)
     (in_bom yes) (on_board yes) (dnp no)
-    (property "Reference" "#PWR0207" (at 215.265 49.53 0)
+    (property "Reference" "#PWR0207" (at 215.265 43.18 0)
       (effects (font (size 1.27 1.27)) hide)
     )
-    (property "Value" "GND" (at 217.805 49.53 0)
+    (property "Value" "GND" (at 217.805 43.18 0)
       (effects (font (size 1 1)))
     )
-    (property "Footprint" "" (at 221.615 49.53 0)
+    (property "Footprint" "" (at 221.615 43.18 0)
       (effects (font (size 1.27 1.27)) hide)
     )
-    (property "Datasheet" "" (at 221.615 49.53 0)
+    (property "Datasheet" "" (at 221.615 43.18 0)
       (effects (font (size 1.27 1.27)) hide)
     )
@@
     )
   )
-  (symbol (lib_id "Connector:Conn_01x10_Pin") (at 226.695 36.83 0) (mirror y) (unit 1)
+  (symbol (lib_id "Connector:Conn_01x10_Pin") (at 226.695 30.48 0) (mirror y) (unit 1)
     (in_bom yes) (on_board yes) (dnp no)
-    (property "Reference" "J27" (at 222.885 50.8 0)
+    (property "Reference" "J27" (at 222.885 44.45 0)
       (effects (font (size 1.27 1.27)) (justify right))
     )
-    (property "Value" "RASP Peripheral" (at 228.6 43.815 90)
+    (property "Value" "RASP Peripheral" (at 228.6 37.465 90)
       (effects (font (size 1 1)) (justify left))
     )
-    (property "Footprint" "Connector_PinHeader_2.54mm:PinHeader_1x10_P2.54mm_Vertical" (at 226.695 36.83 0)
+    (property "Footprint" "Connector_PinHeader_2.54mm:PinHeader_1x10_P2.54mm_Vertical" (at 226.695 30.48 0)
       (effects (font (size 1.27 1.27)) hide)
     )
-    (property "Datasheet" "~" (at 226.695 36.83 0)
+    (property "Datasheet" "~" (at 226.695 30.48 0)
       (effects (font (size 1.27 1.27)) hide)
     )
@@
   (symbol (lib_id "RASPBERRY_PI_4B:RASPBERRY_PI_4B_4GB") (at 64.135 97.79 0) (unit 1)
     (in_bom yes) (on_board yes) (dnp no) (fields_autoplaced)
-    (property "Reference" "U2" (at 64.135 60.325 0)
+    (property "Reference" "U2" (at 64.135 59.69 0)
       (effects (font (size 1.27 1.27)))
     )
-    (property "Value" "RASPBERRY_PI_4B_4GB" (at 64.135 62.865 0)
+    (property "Value" "RASPBERRY_PI_5" (at 64.135 62.23 0)
       (effects (font (size 1.27 1.27)))
     )
@@
     )
   )
-  (symbol (lib_id "power:+3.3V") (at 221.615 26.67 0) (mirror y) (unit 1)
+  (symbol (lib_id "power:+3.3V") (at 221.615 20.32 0) (mirror y) (unit 1)
     (in_bom yes) (on_board yes) (dnp no)
-    (property "Reference" "#PWR0206" (at 221.615 30.48 0)
+    (property "Reference" "#PWR0206" (at 221.615 24.13 0)
       (effects (font (size 1.27 1.27)) hide)
     )
-    (property "Value" "+3.3V" (at 221.615 23.495 0)
+    (property "Value" "+3.3V" (at 221.615 17.145 0)
       (effects (font (size 1 1)))
     )
-    (property "Footprint" "" (at 221.615 26.67 0)
+    (property "Footprint" "" (at 221.615 20.32 0)
       (effects (font (size 1.27 1.27)) hide)
     )
-    (property "Datasheet" "" (at 221.615 26.67 0)
+    (property "Datasheet" "" (at 221.615 20.32 0)
       (effects (font (size 1.27 1.27)) hide)
     )
@@
       (effects (font (size 1.27 1.27)) (justify left bottom))
     )
-    (property "Sheetfile" "soc.kicad_sch" (at 238.125 65.405 0)
+    (property "Sheetfile" "soc.kicad_sch" (at 238.76 70.485 0)
       (effects (font (size 1.27 1.27)) (justify left top))
     )

Commit message: update watch_v3
Parts:
- removed C47, C48: 100uF, Capacitor_SMD:C_0402_1005Metric, symbol Device:C
- added C47, C48: 100uF, Battery:CAPAE830X1000N, symbol UWT1V101MCL1GS:UWT1V101MCL1GS
- J27: footprint Connector_PinHeader_2.54mm:PinHeader_1x10_P2.54mm_Vertical -> Button_Switch_SMD:solder_10
Connections:
- net +3.3V: now also C47.1, C48.1
- net GND: now also C47.2, C48.2
Changed lines of the file:
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@@
     )
   )
-  (symbol (lib_id "Device:C") (at 136.525 184.785 0) (unit 1)
-    (in_bom yes) (on_board yes) (dnp no)
-    (property "Reference" "C48" (at 135.255 186.69 0)
-      (effects (font (size 1 1)) (justify right))
-    )
-    (property "Value" "100uF" (at 142.24 182.88 0)
-      (effects (font (size 1 1)) (justify right))
-    )
-    (property "Footprint" "Capacitor_SMD:C_0402_1005Metric" (at 137.4902 188.595 0)
-      (effects (font (size 1.27 1.27)) hide)
-    )
-    (property "Datasheet" "~" (at 136.525 184.785 0)
-      (effects (font (size 1.27 1.27)) hide)
-    )
-    (pin "1")
-    (pin "2")
-    (instances
-      (project "remote_v2"
-        (path "/06398ea7-2a88-46d2-a66c-c169b1a4e04e"
-          (reference "C48") (unit 1)
-        )
-      )
-    )
-  )
   (symbol (lib_id "power:GND") (at 54.61 21.59 180) (unit 1)
     (in_bom yes) (on_board yes) (dnp no)
@@
       (effects (font (size 1 1)) (justify left))
     )
-    (property "Footprint" "Connector_PinHeader_2.54mm:PinHeader_1x10_P2.54mm_Vertical" (at 226.695 30.48 0)
+    (property "Footprint" "Button_Switch_SMD:solder_10" (at 226.695 30.48 0)
       (effects (font (size 1.27 1.27)) hide)
     )
@@
     )
   )
+  (symbol (lib_id "UWT1V101MCL1GS:UWT1V101MCL1GS") (at 130.175 186.055 270) (unit 1)
+    (in_bom yes) (on_board yes) (dnp no)
+    (property "Reference" "C47" (at 128.27 189.23 0)
+      (effects (font (size 1 1)))
+    )
+    (property "Value" "100uF" (at 126.365 184.785 0)
+      (effects (font (size 1 1)))
+    )
+    (property "Footprint" "Battery:CAPAE830X1000N" (at 130.175 186.055 0)
+      (effects (font (size 1.27 1.27)) (justify bottom) hide)
+    )
+    (property "Datasheet" "" (at 130.175 186.055 0)
+      (effects (font (size 1.27 1.27)) hide)
+    )
+    (property "MF" "Nichicon" (at 130.175 186.055 0)
+      (effects (font (size 1.27 1.27)) (justify bottom) hide)
+    )
+    (property "MAXIMUM_PACKAGE_HEIGHT" "7.7mm" (at 130.175 186.055 0)
+      (effects (font (size 1.27 1.27)) (justify bottom) hide)
+    )
+    (property "Package" "Radial Nichicon" (at 130.175 186.055 0)
+      (effects (font (size 1.27 1.27)) (justify bottom) hide)
+    )
+    (property "Price" "None" (at 130.175 186.055 0)
+      (effects (font (size 1.27 1.27)) (justify bottom) hide)
+    )
+    (property "Check_prices" "https://www.snapeda.com/parts/UWT1V101MCL1GS/Nichicon/view-part/?ref=eda" (at 130.175 186.055 0)
+      (effects (font (size 1.27 1.27)) (justify bottom) hide)
+    )
+    (property "STANDARD" "IPC-7351B" (at 130.175 186.055 0)
+      (effects (font (size 1.27 1.27)) (justify bottom) hide)
+    )
+    (property "PARTREV" "CAT.8100L" (at 130.175 186.055 0)
+      (effects (font (size 1.27 1.27)) (justify bottom) hide)
+    )
+    (property "SnapEDA_Link" "https://www.snapeda.com/parts/UWT1V101MCL1GS/Nichicon/view-part/?ref=snap" (at 130.175 186.055 0)
+      (effects (font (size 1.27 1.27)) (justify bottom) hide)
+    )
+    (property "MP" "UWT1V101MCL1GS" (at 130.175 186.055 0)
+      (effects (font (size 1.27 1.27)) (justify bottom) hide)
+    )
+    (property "Description" "\n                        \n                            Capacitor Aluminum Electrolytic, 1000h 6.3 (Dia.) x 7.7mm, 100uF, 35V, WT Series | Nichicon UWT1V101MCL1GS\n                        \n" (at 130.175 186.055 0)
+      (effects (font (size 1.27 1.27)) (justify bottom) hide)
+    )
+    (property "MANUFACTURER" "Nichicon" (at 130.175 186.055 0)
+      (effects (font (size 1.27 1.27)) (justify bottom) hide)
+    )
+    (property "Availability" "In Stock" (at 130.175 186.055 0)
+      (effects (font (size 1.27 1.27)) (justify bottom) hide)
+    )
+    (property "SNAPEDA_PN" "UWT1V101MCL1GS" (at 130.175 186.055 0)
+      (effects (font (size 1.27 1.27)) (justify bottom) hide)
+    )
+    (pin "1")
+    (pin "2")
+    (instances
+      (project "remote_v2"
+        (path "/06398ea7-2a88-46d2-a66c-c169b1a4e04e"
+          (reference "C47") (unit 1)
+        )
+      )
+    )
+  )
   (symbol (lib_id "power:GND") (at 276.86 116.205 0) (unit 1)
     (in_bom yes) (on_board yes) (dnp no)
@@
     )
   )
+  (symbol (lib_id "UWT1V101MCL1GS:UWT1V101MCL1GS") (at 136.525 186.055 270) (unit 1)
+    (in_bom yes) (on_board yes) (dnp no)
+    (property "Reference" "C48" (at 137.795 187.325 0)
+      (effects (font (size 1 1)))
+    )
+    (property "Value" "100uF" (at 140.335 184.785 0)
+      (effects (font (size 1 1)))
+    )
+    (property "Footprint" "Battery:CAPAE830X1000N" (at 136.525 186.055 0)
+      (effects (font (size 1.27 1.27)) (justify bottom) hide)
+    )
+    (property "Datasheet" "" (at 136.525 186.055 0)
+      (effects (font (size 1.27 1.27)) hide)
+    )
+    (property "MF" "Nichicon" (at 136.525 186.055 0)
+      (effects (font (size 1.27 1.27)) (justify bottom) hide)
+    )
+    (property "MAXIMUM_PACKAGE_HEIGHT" "7.7mm" (at 136.525 186.055 0)
+      (effects (font (size 1.27 1.27)) (justify bottom) hide)
+    )
+    (property "Package" "Radial Nichicon" (at 136.525 186.055 0)
+      (effects (font (size 1.27 1.27)) (justify bottom) hide)
+    )
+    (property "Price" "None" (at 136.525 186.055 0)
+      (effects (font (size 1.27 1.27)) (justify bottom) hide)
+    )
+    (property "Check_prices" "https://www.snapeda.com/parts/UWT1V101MCL1GS/Nichicon/view-part/?ref=eda" (at 136.525 186.055 0)
+      (effects (font (size 1.27 1.27)) (justify bottom) hide)
+    )
+    (property "STANDARD" "IPC-7351B" (at 136.525 186.055 0)
+      (effects (font (size 1.27 1.27)) (justify bottom) hide)
+    )
+    (property "PARTREV" "CAT.8100L" (at 136.525 186.055 0)
+      (effects (font (size 1.27 1.27)) (justify bottom) hide)
+    )
+    (property "SnapEDA_Link" "https://www.snapeda.com/parts/UWT1V101MCL1GS/Nichicon/view-part/?ref=snap" (at 136.525 186.055 0)
+      (effects (font (size 1.27 1.27)) (justify bottom) hide)
+    )
+    (property "MP" "UWT1V101MCL1GS" (at 136.525 186.055 0)
+      (effects (font (size 1.27 1.27)) (justify bottom) hide)
+    )
+    (property "Description" "\n                        \n                            Capacitor Aluminum Electrolytic, 1000h 6.3 (Dia.) x 7.7mm, 100uF, 35V, WT Series | Nichicon UWT1V101MCL1GS\n                        \n" (at 136.525 186.055 0)
+      (effects (font (size 1.27 1.27)) (justify bottom) hide)
+    )
+    (property "MANUFACTURER" "Nichicon" (at 136.525 186.055 0)
+      (effects (font (size 1.27 1.27)) (justify bottom) hide)
+    )
+    (property "Availability" "In Stock" (at 136.525 186.055 0)
+      (effects (font (size 1.27 1.27)) (justify bottom) hide)
+    )
+    (property "SNAPEDA_PN" "UWT1V101MCL1GS" (at 136.525 186.055 0)
+      (effects (font (size 1.27 1.27)) (justify bottom) hide)
+    )
+    (pin "1")
+    (pin "2")
+    (instances
+      (project "remote_v2"
+        (path "/06398ea7-2a88-46d2-a66c-c169b1a4e04e"
+          (reference "C48") (unit 1)
+        )
+      )
+    )
+  )
   (symbol (lib_id "Device:R") (at 113.665 154.305 90) (mirror x) (unit 1)
     (in_bom yes) (on_board yes) (dnp no)
@@
         )
       )
-    )
-  )
-  (symbol (lib_id "Device:C") (at 130.175 184.785 0) (unit 1)
-    (in_bom yes) (on_board yes) (dnp no)
-    (property "Reference" "C47" (at 128.905 186.69 0)
-      (effects (font (size 1 1)) (justify right))
-    )
-    (property "Value" "100uF" (at 130.175 182.88 0)
-      (effects (font (size 1 1)) (justify right))
-    )
-    (property "Footprint" "Capacitor_SMD:C_0402_1005Metric" (at 131.1402 188.595 0)
-      (effects (font (size 1.27 1.27)) hide)
-    )
-    (property "Datasheet" "~" (at 130.175 184.785 0)
-      (effects (font (size 1.27 1.27)) hide)
-    )
-    (pin "1")
-    (pin "2")
-    (instances
-      (project "remote_v2"
-        (path "/06398ea7-2a88-46d2-a66c-c169b1a4e04e"
-          (reference "C47") (unit 1)
-        )
-      )

Commit message: updating watch_v3
Parts:
- removed D11, D12, D8: 1N4148, Diode_SMD:D_SOD-323, symbol SS34:SS34
- removed LS2, LS3, LS4: CMT-8530S-SMT, Capacitor_SMD:CUI_CMT-8530S-SMT, symbol CMT-8530S-SMT:CMT-8530S-SMT
- removed Q5, Q8, Q9: BC847, Package_TO_SOT_SMD:SOT-23, symbol Transistor_BJT:BC847
- added J28: Mode1, Battery:smd_pad_10, symbol Connector:Conn_01x03_Pin
- added J29: Mode3, Battery:smd_pad_10, symbol Connector:Conn_01x03_Pin
- added J30: Mode2, Battery:smd_pad_10, symbol Connector:Conn_01x03_Pin
- added J31: Mode4, Battery:smd_pad_10, symbol Connector:Conn_01x03_Pin
- added R100, R101, R97, R98, R99: 0, Resistor_SMD:R_0402_1005Metric, symbol Device:R
- J25: footprint Button_Switch_SMD:AMASS_XT60-M -> Battery:AMASS_XT60PW-M
Connections:
- net +3.3V: now also R100.1, R98.1; no longer R75.1
- net 5V: now also J25.1 (POS); no longer J25.P (POS)
- net GND: now also J25.2 (NEG), J28.3 (Pin_3), J29.3 (Pin_3), J30.3 (Pin_3), J31.3 (Pin_3); no longer J25.N (NEG)
- net at R75.2: now also J28.2 (Pin_2)
- net at R76.2: now also J29.1 (Pin_1)
- net at R74.2: now also J28.1 (Pin_1)
- new net: J29.2 (Pin_2), R97.2
- new net: J31.1 (Pin_1), R100.2
- new net: J31.2 (Pin_2), R101.2
- new net: J30.2 (Pin_2), R99.2
- new net: J30.1 (Pin_1), R98.2
- new net Mode1: R75.1
- new net Mode2: R99.1
- new net Mode3: R97.1
- new net Mode4: R101.1
Other:
- sheet SoC1 ports: added Mode1, Mode2, Mode3, Mode4; removed BuzzJ2, BuzzJ3, BuzzJ4
- note added: "Mode"
