File: PCB/Remote_V2/remote_v2.kicad_sch (KiCad schematic)
At the start: 100 parts, among them J10 Yaxis J1, J11 Yaxis J2, J12 Yaxis J3, J13 Yaxis J4, J14 ICSP1, J15 ICSP2, J16 ICSP3, J18 Peri Soc 1, J19 Peri Soc 2, J2 ADS1115 A1, J20 Peri Soc 3, J21 UART Soc 1, J22 UART Soc 2, J23 UART Soc 3, J24 5V, J25 XT60-M, J26 UART RASP, J27 RASP Peripheral, J28 Mode1, J29 Mode3, J3 ADS1115 A2, J30 Mode2, J31 Mode4, J4 Xaxis J1, J7 Xaxis J2, J8 Xaxis J3, J9 Xaxis J4, Q4 BC847, SW7 SW_SPDT, SW8 SW_SPDT, U11 Ai-Thinker-Ra-02, U12 Ai-Thinker-Ra-02, U13 MPU-6050, U2 RASPBERRY_PI_5

Commit message: update watch_v3
Parts:
- removed C55, C57: 100uF, Battery:CAPAE830X1000N, symbol UWT1V101MCL1GS:UWT1V101MCL1GS
- removed J14: ICSP1, Button_Switch_SMD:solder_pad_4, symbol Connector:Conn_01x04_Pin
- removed J15: ICSP2, Button_Switch_SMD:solder_pad_4, symbol Connector:Conn_01x04_Pin
- removed J16: ICSP3, Button_Switch_SMD:solder_pad_4, symbol Connector:Conn_01x04_Pin
- added J32, J33, J6: Conn_01x07_Pin, Button_Switch_SMD:solder_7, symbol Connector:Conn_01x07_Pin
- added R10, R15, R8: 0, Resistor_SMD:R_0402_1005Metric, symbol Device:R
Connections:
- net +3.3V: now also J32.6 (Pin_6), J33.6 (Pin_6), J6.6 (Pin_6)
- net EN1: now also J6.4 (Pin_4)
- net EN2: now also J32.4 (Pin_4)
- net EN3: now also J33.4 (Pin_4)
- net GND: now also J32.1 (Pin_1), J33.1 (Pin_1), J6.1 (Pin_1)
- net IO01: now also J6.5 (Pin_5)
- net IO02: now also J32.5 (Pin_5)
- net IO03: now also J33.5 (Pin_5)
- net RX1: now also J6.3 (Pin_3)
- net RX2: now also J32.3 (Pin_3)
- net RX3: now also J33.3 (Pin_3)
- net TX1: now also J6.2 (Pin_2)
- net TX2: now also J32.2 (Pin_2)
- net TX3: now also J33.2 (Pin_2)
- net VCCQ: now also R10.1, R15.1, R8.1
- net ce0: now also J27.8 (Pin_8); no longer J27.5 (Pin_5)
- net ce1: now also J27.9 (Pin_9); no longer J27.6 (Pin_6)
- net miso: now also J27.6 (Pin_6); no longer J27.9 (Pin_9)
- net mosi: now also J27.5 (Pin_5); no longer J27.8 (Pin_8)
- net at U2.1 (3V3): no longer U2.17 (3V3)
- net at U2.2 (5V): no longer U2.4 (5V)
- new net: J33.7 (Pin_7), R15.2
- new net: J6.7 (Pin_7), R8.2
- new net: J32.7 (Pin_7), R10.2
- now unconnected: U2.S1 (SHIELD), U2.S2 (SHIELD), U2.S3 (SHIELD), U2.S4 (SHIELD)
- no-connect marks 39 -> 44
Other:
- removed sheet UART Bridge
- sheet Power Supply ports: added none; removed D1+, D1-, D2+, D2-, D3+, D3-
- note added: "Power Unit"
- note removed: "Power&UART Unit"

Commit message: updating PCBs
Parts:
- removed C45, C46, C49, C50: 0.1uF, Capacitor_SMD:C_0402_1005Metric, symbol Device:C
- removed J18: Peri Soc 1, Button_Switch_SMD:solder_pad_4, symbol Connector:Conn_01x04_Pin
- removed J19: Peri Soc 2, Button_Switch_SMD:solder_pad_4, symbol Connector:Conn_01x04_Pin
- removed J20: Peri Soc 3, Button_Switch_SMD:solder_pad_4, symbol Connector:Conn_01x04_Pin
- removed J21: UART Soc 1, Button_Switch_SMD:solder_pad_4, symbol Connector:Conn_01x04_Pin
- removed J22: UART Soc 2, Button_Switch_SMD:solder_pad_4, symbol Connector:Conn_01x04_Pin
- removed J23: UART Soc 3, Button_Switch_SMD:solder_pad_4, symbol Connector:Conn_01x04_Pin
- removed J27: RASP Peripheral, Button_Switch_SMD:solder_10, symbol Connector:Conn_01x10_Pin
- removed R100, R101, R15, R57, R58, R59, R60, R61, R62, R63, R64, R65, R66, R67, R68, R69, R70, R71, R72, R74, R75, R76, R77, R78, R90, R97, R98, R99: 0, Resistor_SMD:R_0402_1005Metric, symbol Device:R
- added R1: 0, Resistor_SMD:R_0402_1005Metric, symbol Device:R
- R93, R94: value 220 -> 4.7K
- U13: footprint Button_Switch_SMD:QFN50P400X400X95-24N -> Package_DFN_QFN:QFN-24-1EP_3x3mm_P0.4mm_EP1.75x1.6mm
Connections:
- net +3.3V: now also D13.2 (A), D14.2 (A), J10.1 (Pin_1), J11.1 (Pin_1), J12.1 (Pin_1), J13.1 (Pin_1), J28.1 (Pin_1), J29.1 (Pin_1), J30.1 (Pin_1), J31.1 (Pin_1), J4.1 (Pin_1), J7.1 (Pin_1), J8.1 (Pin_1), J9.1 (Pin_1)
- net GND: no longer D13.1 (K), D14.1 (K)
- net Mode1: now also J28.2 (Pin_2)
- net Mode2: now also J30.2 (Pin_2)
- net Mode3: now also J29.2 (Pin_2)
- net Mode4: now also J31.2 (Pin_2)
- net VCCQ: now also R1.1
- net Vx1: now also J4.2 (Pin_2)
- net Vx2: now also J7.2 (Pin_2)
- net Vx3: now also J8.2 (Pin_2)
- net Vx4: now also J9.2 (Pin_2)
- net Vy1: now also J10.2 (Pin_2)
- net Vy2: now also J11.2 (Pin_2)
- net Vy3: now also J12.2 (Pin_2)
- net Vy4: now also J13.2 (Pin_2)
- net at J33.7 (Pin_7): now also R1.2
- net at U13.21 (RESV), U13.22 (RESV): no longer U13.19 (RESV)
- net at R94.1: now also D14.1 (K); no longer D14.2 (A)
- net at R93.2: now also D13.1 (K); no longer D13.2 (A)
- net ce0: no longer names the net of U2.24 (GPIO8/~{SPI_CE0})
- net ce1: no longer names the net of U2.26 (GPIO7/~{SPI_CE1})
- net gp17: no longer names the net of U2.11 (GPIO17/GPIO_GEN0)
- net gp18: no longer names the net of U2.12 (GPIO18/GPIO_GEN1)
- net gp27: no longer names the net of U2.13 (GPIO27/GPIO_GEN2)
- net miso: no longer names the net of U2.21 (GPIO9/SPI_MISO)
- net mosi: no longer names the net of U2.19 (GPIO10/SPI_MOSI)
- net sclk: no longer names the net of U2.23 (GPIO11/SPI_SCLK)
- now unconnected: U13.14 (NC), U13.15 (NC), U13.16 (NC), U13.17 (NC), U13.2 (NC), U13.3 (NC), U13.4 (NC), U13.5 (NC)
- no-connect marks 44 -> 59
Other:
- sheet SoC1 ports: added none; removed RX_2, RX_3, RX_4, S1-12, S1-13, S1-14, S2-26, S2-27, S2-32, S3-13, S3-14, S3-15, TX_2, TX_3
- note added: "UART Rasp-Port"
- note removed: "Peri. RASPI"
- note removed: "Peripheral Port"
- note removed: "UART1 PORT"
- moved on the sheet: C39, C40, C41, C42, C43, C44, D13, D14, J24, J25, J26, R93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
