File: PCB/Remote_V2/soc.kicad_sch (KiCad schematic)
At the start: 35 parts, among them SW1 SW_DPST_x2, SW2 SW_DPST_x2, SW3 SW_DPST_x2, SW4 SW_DPST_x2, SW5 SW_DPST_x2, SW6 SW_DPST_x2, U10 ESP32-WROOM-32D, U6 ESP32-WROOM-32D, U8 ESP32-WROOM-32D

Commit message: remote_v2 update
Parts:
- removed C24, C25, C26, C27, C28, C29, C33, C34, C35: 0.1uF, Capacitor_SMD:C_0402_1005Metric, symbol Device:C
- removed R22, R23: 1K, Resistor_SMD:R_0402_1005Metric, symbol Device:R
- removed U10, U6, U8: ESP32-WROOM-32D, RF_Module:ESP32-WROOM-32D, symbol RF_Module:ESP32-WROOM-32D
- added C89, C90, C91, C92, C93, C94, C95, C96, C97: 0.1uF, Capacitor_SMD:C_0402_1005Metric, symbol Device:C
- added R95: 0, Resistor_SMD:R_0402_1005Metric, symbol Device:R
- added R96: 1K, Resistor_SMD:R_0402_1005Metric, symbol Device:R
- added U22, U23, U24: ESP32-WROOM-32D, RF_Module:ESP32-WROOM-32D, symbol RF_Module:ESP32-WROOM-32D
- R25, R30, R48: value 0 -> 1K
- R27, R38: value 1K -> 0
Connections:
- net +3.3V: now also R25.1, R28.2, R31.1, R33.1, R34.2, R50.1, R51.2, R95.2, R96.2; no longer R25.2, R28.1, R31.2, R33.2, R34.1, R50.2, R51.1
- net Aa: now also U23.37 (IO23)
- net Ab: now also U23.10 (IO25)
- net BuzzJ1: now also U23.29 (IO5)
- net BuzzJ2: now also U23.14 (IO12)
- net BuzzJ3: now also U23.16 (IO13)
- net BuzzJ4: now also U23.13 (IO14)
- net DIO11: now also U24.24 (IO2)
- net DIO12: now also U24.26 (IO4)
- net EN1: now also R26.1, C89.2, U22.3 (EN); no longer R24.1
- net EN2: now also R34.1, C92.2, U23.3 (EN); no longer R29.1
- net EN3: now also R51.1, C95.2, U24.3 (EN); no longer R38.1
- net GND: now also C89.1, C90.1, C91.1, C92.1, C93.1, C94.1, C95.1, C96.1, C97.1, U22.1 (GND), U22.15 (GND), U22.38 (GND), U22.39 (GND), U23.1 (GND), U23.15 (GND), U23.38 (GND), U23.39 (GND), U24.1 (GND), U24.15 (GND), U24.38 (GND), U24.39 (GND)
- net IO01: now also R28.1, C91.2, U22.25 (IO0); no longer R26.1
- net IO02: now also R48.1, C94.2, U23.25 (IO0); no longer R31.1
- net IO03: now also C97.2, R96.1, U24.25 (IO0); no longer R49.1
- net RST1: now also U24.10 (IO25)
- net RST2: now also U24.11 (IO26)
- net RX1: now also U22.35 (TXD0/IO1)
- net RX2: now also U23.35 (TXD0/IO1)
- net RX3: now also U24.35 (TXD0/IO1)
- net RX_2: now also U22.27 (IO16)
- net RX_3: now also U23.27 (IO16)
- net RX_4: now also U24.27 (IO16)
- net S1-12: now also U22.14 (IO12)
- net S1-13: now also U22.16 (IO13)
- net S1-14: now also U22.13 (IO14)
- net S2-26: now also U23.11 (IO26)
- net S2-27: now also U23.12 (IO27)
- net S2-32: now also U23.8 (IO32)
- net S3-13: now also U24.16 (IO13)
- net S3-14: now also U24.13 (IO14)
- net S3-15: now also U24.23 (IO15)
- net SCL1: now also R25.2, U22.36 (IO22)
- net SCL2: now also R31.2, U23.36 (IO22); no longer R28.2
- net SCL3: now also R50.2, U24.36 (IO22); no longer R34.2
- net SCLx: now also R33.2, U23.31 (IO19); no longer R50.1
- net SDA1: now also R24.1, U22.33 (IO21)
- net SDA2: now also R29.1, U23.33 (IO21); no longer R27.1
- net SDA3: now also R49.1, U24.33 (IO21); no longer R33.1
- net SDAx: now also R30.1, U23.30 (IO18); no longer R51.2
- net TX1: now also U22.34 (RXD0/IO3)
- net TX2: now also U23.34 (RXD0/IO3)
- net TX3: now also U24.34 (RXD0/IO3)
- net TX_2: now also U22.28 (IO17)
- net TX_3: now also U23.28 (IO17)
- net TX_4: now also U24.28 (IO17)
- net VCS_1: now also U24.29 (IO5)
- net VCS_2: now also U24.14 (IO12)
- net VMISO: now also U24.31 (IO19)
- net VMOSI: now also U24.37 (IO23)
- net VSCK: now also U24.30 (IO18)
- new net: C93.2, R38.1, U23.2 (VDD)
- new net: C90.2, R27.1, U22.2 (VDD)
- new net: C96.2, R95.1, U24.2 (VDD)
Other:
- note added: "ESP 32"
- note added: "H"
- note added: "SoC 1"
- note added: "SoC 2"
- note added: "SoC 3"
- note removed: "1"
- note removed: "2"
- note removed: "SoC"
- company: (none) -> Dharma Bot KRS
- title: (none) -> SoC_RemoteV2

Commit message: updating watch_v3
Connections:
- net Mode4: now reaches U23.23 (IO15)
- net BuzzJ2 renamed Mode1
- net BuzzJ3 renamed Mode2
- net BuzzJ4 renamed Mode3
- no-connect marks 49 -> 48
Changed lines of the file:
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@@
   (no_connect (at 85.725 125.095))
   (no_connect (at 85.725 109.855))
-  (no_connect (at 169.545 92.075))
   (no_connect (at 254 127.635))
   (no_connect (at 139.065 109.855))
@@
     (effects (font (size 1.27 1.27)) (justify left bottom))
   )
-  (label "BuzzJ3" (at 169.545 86.995 0) (fields_autoplaced)
+  (label "Mode2" (at 169.545 86.995 0) (fields_autoplaced)
     (effects (font (size 1 1)) (justify left bottom))
   )
@@
     (effects (font (size 1.27 1.27)) (justify left bottom))
   )
-  (label "BuzzJ4" (at 169.545 89.535 0) (fields_autoplaced)
+  (label "Mode3" (at 169.545 89.535 0) (fields_autoplaced)
     (effects (font (size 1 1)) (justify left bottom))
   )
@@
     (effects (font (size 1.27 1.27)) (justify left bottom))
   )
+  (label "Mode2" (at 73.66 174.625 90) (fields_autoplaced)
+    (effects (font (size 1 1)) (justify left bottom))
+  )
   (label "S1-13" (at 52.705 162.56 90) (fields_autoplaced)
     (effects (font (size 1 1)) (justify left bottom))
@@
     (effects (font (size 1 1)) (justify left bottom))
   )
-  (label "BuzzJ2" (at 70.485 174.625 90) (fields_autoplaced)
-    (effects (font (size 1 1)) (justify left bottom))
-  )
   (label "DIO11" (at 31.75 186.69 90) (fields_autoplaced)
     (effects (font (size 1 1)) (justify left bottom))
@@
     (effects (font (size 1 1)) (justify left bottom))
   )
+  (label "Mode1" (at 70.485 174.625 90) (fields_autoplaced)
+    (effects (font (size 1 1)) (justify left bottom))
+  )
   (label "IO02" (at 36.195 162.56 90) (fields_autoplaced)
     (effects (font (size 1.27 1.27)) (justify left bottom))
-  )
-  (label "BuzzJ4" (at 78.105 174.625 90) (fields_autoplaced)
-    (effects (font (size 1 1)) (justify left bottom))
   )
   (label "TX_2" (at 85.725 97.155 0) (fields_autoplaced)
@@
     (effects (font (size 1.27 1.27)) (justify left bottom))
   )
+  (label "Mode4" (at 79.375 174.625 90) (fields_autoplaced)
+    (effects (font (size 1 1)) (justify left bottom))
+  )
   (label "DIO12" (at 254 79.375 0) (fields_autoplaced)
     (effects (font (size 1 1)) (justify left bottom))
@@
     (effects (font (size 1 1)) (justify left bottom))
   )
-  (label "BuzzJ2" (at 169.545 84.455 0) (fields_autoplaced)
+  (label "Mode1" (at 169.545 84.455 0) (fields_autoplaced)
     (effects (font (size 1 1)) (justify left bottom))
   )
@@
   )
   (label "S2-32" (at 169.545 120.015 0) (fields_autoplaced)
+    (effects (font (size 1 1)) (justify left bottom))
+  )
+  (label "Mode3" (at 76.835 174.625 90) (fields_autoplaced)
+    (effects (font (size 1 1)) (justify left bottom))
+  )
+  (label "Mode4" (at 169.545 92.075 0) (fields_autoplaced)
     (effects (font (size 1 1)) (justify left bottom))
   )
@@
     (effects (font (size 1 1)) (justify left bottom))
   )
-  (label "BuzzJ3" (at 74.295 174.625 90) (fields_autoplaced)
-    (effects (font (size 1 1)) (justify left bottom))
-  )
   (label "VSCK" (at 254 99.695 0) (fields_autoplaced)
     (effects (font (size 1 1)) (justify left bottom))
@@
     (effects (font (size 1 1)) (justify right))
   )
-  (hierarchical_label "BuzzJ3" (shape input) (at 74.295 174.625 270) (fields_autoplaced)
-    (effects (font (size 1 1)) (justify right))
-  )
   (hierarchical_label "S3-14" (shape input) (at 46.355 186.69 270) (fields_autoplaced)
     (effects (font (size 1 1)) (justify right))
@@
     (effects (font (size 1 1)) (justify right))
   )
-  (hierarchical_label "BuzzJ4" (shape input) (at 78.105 174.625 270) (fields_autoplaced)
-    (effects (font (size 1 1)) (justify right))
-  )
   (hierarchical_label "SCL2" (shape input) (at 43.18 174.625 270) (fields_autoplaced)
     (effects (font (size 1 1)) (justify right))
@@
     (effects (font (size 1 1)) (justify right))
   )
+  (hierarchical_label "Mode2" (shape input) (at 73.66 174.625 270) (fields_autoplaced)
+    (effects (font (size 1 1)) (justify right))
+  )
   (hierarchical_label "TX2" (shape input) (at 26.67 162.56 270) (fields_autoplaced)
     (effects (font (size 1 1)) (justify right))
@@
     (effects (font (size 1 1)) (justify right))
   )
-  (hierarchical_label "BuzzJ2" (shape input) (at 70.485 174.625 270) (fields_autoplaced)
+  (hierarchical_label "Mode1" (shape input) (at 70.485 174.625 270) (fields_autoplaced)
     (effects (font (size 1 1)) (justify right))
   )
@@
     (effects (font (size 1 1)) (justify right))
   )
+  (hierarchical_label "Mode4" (shape input) (at 79.375 174.625 270) (fields_autoplaced)
+    (effects (font (size 1 1)) (justify right))
+  )
   (hierarchical_label "SCL3" (shape input) (at 90.805 186.055 270) (fields_autoplaced)
     (effects (font (size 1 1)) (justify right))
@@
     (effects (font (size 1 1)) (justify right))
   )
+  (hierarchical_label "Mode3" (shape input) (at 76.835 174.625 270) (fields_autoplaced)
+    (effects (font (size 1 1)) (justify right))
+  )

Commit message: updating PCBs
Parts:
- removed R29, R31, R49, R50: 1K, Resistor_SMD:R_0402_1005Metric, symbol Device:R
- R24, R25, R26, R28, R30, R33, R34, R48, R51, R96: value 1K -> 10K
- SW1, SW2, SW3, SW4, SW5, SW6: footprint Button_Switch_SMD:SW_Tactile_SPST_NO_Straight_CK_PTS636Sx25SMTRLFS -> Button_Switch_SMD:SW_SPST_B3U-1000P-B
Connections:
- net RX_2: no longer names the net of U22.27 (IO16)
- net RX_3: no longer names the net of U23.27 (IO16)
- net RX_4: no longer names the net of U24.27 (IO16)
- net S1-12: no longer names the net of U22.14 (IO12)
- net S1-13: no longer names the net of U22.16 (IO13)
- net S1-14: no longer names the net of U22.13 (IO14)
- net S2-26: no longer names the net of U23.11 (IO26)
- net S2-27: no longer names the net of U23.12 (IO27)
- net S2-32: no longer names the net of U23.8 (IO32)
- net S3-13: no longer names the net of U24.16 (IO13)
- net S3-14: no longer names the net of U24.13 (IO14)
- net S3-15: no longer names the net of U24.23 (IO15)
- net TX_2: no longer names the net of U22.28 (IO17)
- net TX_3: no longer names the net of U23.28 (IO17)
- net TX_4: no longer names the net of U24.28 (IO17)
- no-connect marks 48 -> 63
