File: PCB/Remote_V2/power_supply.kicad_sch (KiCad schematic)
At the start: 69 parts, among them J1 USB_C_Receptacle_USB2.0_16P, J5 USB_C_Receptacle_USB2.0_16P, J6 USB_C_Receptacle_USB2.0_16P, Q1 AO3401A, Q2 AO3401A, Q3 AO3401A, U1 AMS1117-3.3, U3 AMS1117-3.3, U4 AMS1117-3.3, U5 AMS1117-3.3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

Commit message: remote_v2 update
Other:
- note added: "H"
- note added: "POWER UNIT"
- company: (none) -> KRS_Dharma_bot
- title: (none) -> USB-Power unit
Changed lines of the file:
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@@
 (kicad_sch (version 20230121) (generator eeschema)
   (paper "A4")
+  (title_block
+    (title "USB-Power unit")
+    (date "2024-11-28")
+    (rev "V2")
+    (company "KRS_Dharma_bot")
+  )
   (junction (at 142.24 74.93) (diameter 0) (color 0 0 0 0)
   )
@@
     (stroke (width 0) (type default))
   )
+  (rectangle (start 156.21 132.715) (end 205.74 164.465)
+    (stroke (width 0.3) (type dash) (color 255 16 12 1))
+    (fill (type none))
+  )
   (rectangle (start 156.21 63.5) (end 276.86 129.54)
     (stroke (width 0.3) (type dash) (color 255 16 12 1))
@@
     (fill (type none))
   )
+  (text "POWER UNIT\n" (at 189.23 45.085 0)
+    (effects (font (size 6 6) (thickness 1.6) bold (color 253 61 255 1)) (justify left bottom))
+  )
+  (text "H\n" (at 200.025 136.525 0)
+    (effects (font (size 2 2) (thickness 0.4) bold) (justify left bottom))
+  )
   (text "Power System\n" (at 254.635 67.31 0)
     (effects (font (size 2 2) (thickness 0.4) bold) (justify left bottom))
@@
     (effects (font (size 1.27 1.27)) (justify left bottom))
   )
+  (label "D1-" (at 168.91 139.065 0) (fields_autoplaced)
+    (effects (font (size 1.27 1.27)) (justify left bottom))
+  )
+  (label "D3-" (at 193.04 139.065 0) (fields_autoplaced)
+    (effects (font (size 1.27 1.27)) (justify left bottom))
+  )
+  (label "D2-" (at 180.34 139.065 0) (fields_autoplaced)
+    (effects (font (size 1.27 1.27)) (justify left bottom))
+  )
+  (label "D2+" (at 173.99 139.065 0) (fields_autoplaced)
+    (effects (font (size 1.27 1.27)) (justify left bottom))
+  )
+  (label "D3+" (at 186.055 139.065 0) (fields_autoplaced)
+    (effects (font (size 1.27 1.27)) (justify left bottom))
+  )
   (label "D2-" (at 60.96 139.065 0) (fields_autoplaced)
     (effects (font (size 1.27 1.27)) (justify left bottom))
@@
     (effects (font (size 1.27 1.27)) (justify left bottom))
   )
+  (label "D1+" (at 163.195 139.065 0) (fields_autoplaced)
+    (effects (font (size 1.27 1.27)) (justify left bottom))
+  )
   (label "D3+" (at 187.325 106.68 0) (fields_autoplaced)
     (effects (font (size 1.27 1.27)) (justify left bottom))
   )
+  (hierarchical_label "5V" (shape input) (at 173.355 154.305 270) (fields_autoplaced)
+    (effects (font (size 1 1)) (justify right))
+  )
+  (hierarchical_label "D3-" (shape input) (at 193.04 139.065 270) (fields_autoplaced)
+    (effects (font (size 1 1)) (justify right))
+  )
+  (hierarchical_label "D2+" (shape input) (at 173.99 139.065 270) (fields_autoplaced)
+    (effects (font (size 1 1)) (justify right))
+  )
+  (hierarchical_label "3.3V" (shape input) (at 177.8 154.305 270) (fields_autoplaced)
+    (effects (font (size 1 1)) (justify right))
+  )
+  (hierarchical_label "GND" (shape input) (at 182.88 153.035 0) (fields_autoplaced)
+    (effects (font (size 1 1)) (justify left))
+  )
+  (hierarchical_label "VCCQ" (shape input) (at 168.275 154.305 270) (fields_autoplaced)
+    (effects (font (size 1 1)) (justify right))
+  )
+  (hierarchical_label "D3+" (shape input) (at 186.055 139.065 270) (fields_autoplaced)
+    (effects (font (size 1 1)) (justify right))
+  )
+  (hierarchical_label "VBUS" (shape input) (at 163.195 154.305 270) (fields_autoplaced)
+    (effects (font (size 1 1)) (justify right))
+  )
+  (hierarchical_label "D1-" (shape input) (at 168.91 139.065 270) (fields_autoplaced)
+    (effects (font (size 1 1)) (justify right))
+  )
+  (hierarchical_label "D2-" (shape input) (at 180.34 139.065 270) (fields_autoplaced)
+    (effects (font (size 1 1)) (justify right))
+  )
+  (hierarchical_label "D1+" (shape input) (at 163.195 139.065 270) (fields_autoplaced)
+    (effects (font (size 1 1)) (justify right))
+  )
   (symbol (lib_id "Device:C") (at 125.095 71.12 0) (unit 1)
     (in_bom yes) (on_board yes) (dnp no)
@@
     )
   )
+  (symbol (lib_id "power:GND") (at 182.88 153.035 0) (unit 1)
+    (in_bom yes) (on_board yes) (dnp no)
+    (property "Reference" "#PWR0212" (at 182.88 159.385 0)
+      (effects (font (size 1.27 1.27)) hide)
+    )
+    (property "Value" "GND" (at 182.88 156.845 0)
+      (effects (font (size 1 1)))
+    )
+    (property "Footprint" "" (at 182.88 153.035 0)
+      (effects (font (size 1.27 1.27)) hide)
+    )
+    (property "Datasheet" "" (at 182.88 153.035 0)
+      (effects (font (size 1.27 1.27)) hide)
+    )
+    (pin "1")
+    (instances
+      (project "remote_v2"
+        (path "/06398ea7-2a88-46d2-a66c-c169b1a4e04e/3b6afdb5-b9e5-4027-9a2f-f8f9d1d3e58a"
+          (reference "#PWR0212") (unit 1)
+        )
+      )
+    )
+  )
   (symbol (lib_id "power:VBUS") (at 93.98 53.34 0) (unit 1)
     (in_bom yes) (on_board yes) (dnp no)
@@
   (symbol (lib_id "Device:R") (at 198.12 98.425 0) (unit 1)
     (in_bom yes) (on_board yes) (dnp no)
-    (property "Reference" "R17" (at 194.945 100.33 0)
+    (property "Reference" "R17" (at 196.85 95.885 90)
       (effects (font (size 1 1)) (justify left))
     )
@@
     )
   )
+  (symbol (lib_id "power:VBUS") (at 163.195 154.305 0) (unit 1)
+    (in_bom yes) (on_board yes) (dnp no)
+    (property "Reference" "#PWR0211" (at 163.195 158.115 0)
+      (effects (font (size 1.27 1.27)) hide)
+    )
+    (property "Value" "VBUS" (at 163.195 151.13 0)
+      (effects (font (size 1 1)))
+    )
+    (property "Footprint" "" (at 163.195 154.305 0)
+      (effects (font (size 1.27 1.27)) hide)
+    )
+    (property "Datasheet" "" (at 163.195 154.305 0)
+      (effects (font (size 1.27 1.27)) hide)
+    )
+    (pin "1")
+    (instances
+      (project "remote_v2"
+        (path "/06398ea7-2a88-46d2-a66c-c169b1a4e04e/3b6afdb5-b9e5-4027-9a2f-f8f9d1d3e58a"
+          (reference "#PWR0211") (unit 1)
+        )
+      )
+    )
+  )
   (symbol (lib_id "Device:R") (at 67.31 65.405 0) (unit 1)
     (in_bom yes) (on_board yes) (dnp no)
@@
     )
   )
+  (symbol (lib_id "power:+3.3V") (at 177.8 154.305 0) (unit 1)
+    (in_bom yes) (on_board yes) (dnp no)
+    (property "Reference" "#PWR0210" (at 177.8 158.115 0)
+      (effects (font (size 1.27 1.27)) hide)
+    )
+    (property "Value" "+3.3V" (at 177.8 151.13 0)
+      (effects (font (size 1 1)))
+    )
+    (property "Footprint" "" (at 177.8 154.305 0)
+      (effects (font (size 1.27 1.27)) hide)
+    )
+    (property "Datasheet" "" (at 177.8 154.305 0)
+      (effects (font (size 1.27 1.27)) hide)
+    )
+    (pin "1")
+    (instances
+      (project "remote_v2"
+        (path "/06398ea7-2a88-46d2-a66c-c169b1a4e04e/3b6afdb5-b9e5-4027-9a2f-f8f9d1d3e58a"
+          (reference "#PWR0210") (unit 1)
+        )
+      )
+    )
+  )
   (symbol (lib_id "Connector:USB_C_Receptacle_USB2.0_16P") (at 172.085 101.6 0) (unit 1)
     (in_bom yes) (on_board yes) (dnp no) (fields_autoplaced)
@@
     )
   )
+  (symbol (lib_id "power:VCCQ") (at 168.275 154.305 0) (unit 1)
+    (in_bom yes) (on_board yes) (dnp no)
+    (property "Reference" "#PWR0209" (at 168.275 158.115 0)
+      (effects (font (size 1.27 1.27)) hide)
+    )
+    (property "Value" "VCCQ" (at 168.275 151.13 0)
+      (effects (font (size 1 1)))
+    )
+    (property "Footprint" "" (at 168.275 154.305 0)
+      (effects (font (size 1.27 1.27)) hide)
+    )
+    (property "Datasheet" "" (at 168.275 154.305 0)
+      (effects (font (size 1.27 1.27)) hide)
+    )
+    (pin "1")
+    (instances
+      (project "remote_v2"
+        (path "/06398ea7-2a88-46d2-a66c-c169b1a4e04e/3b6afdb5-b9e5-4027-9a2f-f8f9d1d3e58a"
+          (reference "#PWR0209") (unit 1)
+        )
+      )
+    )
+  )
   (symbol (lib_id "power:GND") (at 85.09 64.77 0) (unit 1)
     (in_bom yes) (on_board yes) (dnp no)
@@
         )
       )
+    )
+  )
+  (symbol (lib_id "power:+5V") (at 173.355 154.305 0) (unit 1)
+    (in_bom yes) (on_board yes) (dnp no)
+    (property "Reference" "#PWR0208" (at 173.355 158.115 0)
+      (effects (font (size 1.27 1.27)) hide)
+    )
+    (property "Value" "+5V" (at 173.355 150.495 0)
+      (effects (font (size 1 1)))
+    )
+    (property "Footprint" "" (at 173.355 154.305 0)
+      (effects (font (size 1.27 1.27)) hide)
+    )
+    (property "Datasheet" "" (at 173.355 154.305 0)
+      (effects (font (size 1.27 1.27)) hide)
+    )
+    (pin "1")
+    (instances
+      (project "remote_v2"
+        (path "/06398ea7-2a88-46d2-a66c-c169b1a4e04e/3b6afdb5-b9e5-4027-9a2f-f8f9d1d3e58a"
+          (reference "#PWR0208") (unit 1)
+        )
+      )

Commit message: update watch_v3
Parts:
- removed J1, J5, J6: USB_C_Receptacle_USB2.0_16P, Connector_USB:USB_C_Receptacle_GCT_USB4105-xx-A_16P_TopMnt_Horizontal, symbol Connector:USB_C_Receptacle_USB2.0_16P
- removed R1, R10, R15, R17, R3, R8: 5.1K, Resistor_SMD:R_0402_1005Metric, symbol Device:R
Connections:
- no-connect marks 6 -> 0
Other:
- moved on the sheet: C1, C10, C11, C12, C13, C14, C15, C16, C17, C18, C19, C2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

Commit message: updating PCBs
Parts:
- removed C1, C11, C12, C13, C14, C15, C16, C17, C18, C19, C20, C21, C22, C23, C63, C64, C65, C66, C67, C68, C69: 0.1uF, Capacitor_SMD:C_0402_1005Metric, symbol Device:C
- removed D3, D5: SS34, Button_Switch_SMD:P25_DO-214AC_SMA, symbol SS34:SS34
- removed D4, D6: LED, LED_SMD:LED_0402_1005Metric, symbol Device:LED
- removed Q2, Q3: AO3401A, Package_TO_SOT_SMD:SOT-23, symbol Transistor_FET:AO3401A
- removed R11, R18: 100K, Resistor_SMD:R_0402_1005Metric, symbol Device:R
- removed R12, R13, R16, R19, R20, R9: 0, Resistor_SMD:R_0402_1005Metric, symbol Device:R
- removed R14, R21: 150E, Resistor_SMD:R_0402_1005Metric, symbol Device:R
- removed U5, U7: AMS1117-3.3, Package_TO_SOT_SMD:SOT-223-3_TabPin2, symbol Regulator_Linear:AMS1117-3.3
Connections:
- net at U3.2 (VO), U4.2 (VO): now also R6.2, U1.2 (VO), U9.2 (VO)
Other:
- note removed: "ESP-2"
- note removed: "ESP-3"

Commit message: updating PCB design
Parts:
- added R3: 0, Resistor_SMD:R_0402_1005Metric, symbol Device:R
Connections:
- net +5V: now also R3.1
- net VBUS: now also C3.2, R3.2
- net at D1.C, Q1.3 (D), R5.2: no longer C3.2
Changed lines of the file:
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@@
   (junction (at 108.585 72.39) (diameter 0) (color 0 0 0 0)
   )
+  (junction (at 73.025 41.275) (diameter 0) (color 0 0 0 0)
+  )
   (junction (at 99.695 58.42) (diameter 0) (color 0 0 0 0)
   )
@@
     (stroke (width 0) (type default))
   )
-  (wire (pts (xy 73.025 58.42) (xy 73.025 62.23))
+  (wire (pts (xy 76.2 43.815) (xy 76.2 41.275))
+    (stroke (width 0) (type default))
+  )
+  (wire (pts (xy 83.82 43.815) (xy 83.82 58.42))
+    (stroke (width 0) (type default))
+  )
+  (wire (pts (xy 74.295 62.23) (xy 80.645 62.23))
     (stroke (width 0) (type default))
   )
@@
     (stroke (width 0) (type default))
   )
+  (wire (pts (xy 73.025 40.64) (xy 73.025 41.275))
+    (stroke (width 0) (type default))
+  )
   (wire (pts (xy 99.06 75.565) (xy 99.695 75.565))
     (stroke (width 0) (type default))
@@
     (stroke (width 0) (type default))
   )
-  (wire (pts (xy 73.025 62.23) (xy 74.295 62.23))
-    (stroke (width 0) (type default))
-  )
   (wire (pts (xy 62.865 46.99) (xy 65.405 46.99))
     (stroke (width 0) (type default))
@@
     (stroke (width 0) (type default))
   )
+  (wire (pts (xy 80.645 58.42) (xy 80.645 62.23))
+    (stroke (width 0) (type default))
+  )
   (wire (pts (xy 83.82 93.345) (xy 83.82 111.125))
     (stroke (width 0) (type default))
@@
     (stroke (width 0) (type default))
   )
+  (wire (pts (xy 76.2 41.275) (xy 73.025 41.275))
+    (stroke (width 0) (type default))
+  )
   (wire (pts (xy 108.585 58.42) (xy 107.315 58.42))
     (stroke (width 0) (type default))
@@
   )
   (wire (pts (xy 62.23 58.42) (xy 62.865 58.42))
+    (stroke (width 0) (type default))
+  )
+  (wire (pts (xy 73.025 41.275) (xy 73.025 41.91))
     (stroke (width 0) (type default))
   )
@@
     )
   )
-  (symbol (lib_id "power:+5V") (at 73.025 41.91 0) (unit 1)
-    (in_bom yes) (on_board yes) (dnp no)
-    (property "Reference" "#PWR069" (at 73.025 45.72 0)
-      (effects (font (size 1.27 1.27)) hide)
-    )
-    (property "Value" "+5V" (at 73.025 38.1 0)
-      (effects (font (size 1 1)))
-    )
-    (property "Footprint" "" (at 73.025 41.91 0)
-      (effects (font (size 1.27 1.27)) hide)
-    )
-    (property "Datasheet" "" (at 73.025 41.91 0)
+  (symbol (lib_id "power:+5V") (at 73.025 40.64 0) (unit 1)
+    (in_bom yes) (on_board yes) (dnp no)
+    (property "Reference" "#PWR069" (at 73.025 44.45 0)
+      (effects (font (size 1.27 1.27)) hide)
+    )
+    (property "Value" "+5V" (at 73.025 36.83 0)
+      (effects (font (size 1 1)))
+    )
+    (property "Footprint" "" (at 73.025 40.64 0)
+      (effects (font (size 1.27 1.27)) hide)
+    )
+    (property "Datasheet" "" (at 73.025 40.64 0)
       (effects (font (size 1.27 1.27)) hide)
     )
@@
         )
       )
+    )
+  )
+  (symbol (lib_id "Device:R") (at 80.01 43.815 90) (unit 1)
+    (in_bom yes) (on_board yes) (dnp no)
+    (property "Reference" "R3" (at 81.28 45.72 90)
+      (effects (font (size 1 1)) (justify left))
+    )
+    (property "Value" "0" (at 80.645 43.815 90)
+      (effects (font (size 1 1)) (justify left))
+    )
+    (property "Footprint" "Resistor_SMD:R_0402_1005Metric" (at 80.01 45.593 90)
+      (effects (font (size 1.27 1.27)) hide)
+    )
+    (property "Datasheet" "~" (at 80.01 43.815 0)
+      (effects (font (size 1.27 1.27)) hide)
+    )
+    (pin "1")
+    (pin "2")
+    (instances
+      (project "remote_v2"
+        (path "/06398ea7-2a88-46d2-a66c-c169b1a4e04e/3b6afdb5-b9e5-4027-9a2f-f8f9d1d3e58a"
+          (reference "R3") (unit 1)
+        )
+      )
